Commit message: fixes

File: sensorob_description/urdf/sensorob.xacro (robot description, xacro)
@@ -24,5 +24,5 @@
   </collision>
 </link>
-<link name="link_1_1">
+<link name="link_1">
   <inertial>
     <origin xyz="-0.017391128474433415 -0.007793862548282313 0.09170345730211693" rpy="0 0 0"/>
@@ -33,5 +33,5 @@
     <origin xyz="-0.06828 -0.001091 -0.070444" rpy="0 0 0"/>
     <geometry>
-      <mesh filename="package://sensorob_description/meshes/link_1_1.stl" scale="0.001 0.001 0.001"/>
+      <mesh filename="package://sensorob_description/meshes/link_1.stl" scale="0.001 0.001 0.001"/>
     </geometry>
     <material name="silver"/>
@@ -40,9 +40,9 @@
     <origin xyz="-0.06828 -0.001091 -0.070444" rpy="0 0 0"/>
     <geometry>
-      <mesh filename="package://sensorob_description/meshes/link_1_1.stl" scale="0.001 0.001 0.001"/>
+      <mesh filename="package://sensorob_description/meshes/link_1.stl" scale="0.001 0.001 0.001"/>
     </geometry>
   </collision>
 </link>
-<link name="link_2_1">
+<link name="link_2">
   <inertial>
     <origin xyz="-0.03597352078588314 -0.017962304231270702 0.2436907782754546" rpy="0 0 0"/>
@@ -53,5 +53,5 @@
     <origin xyz="0.023626 0.041765 -0.187444" rpy="0 0 0"/>
     <geometry>
-      <mesh filename="package://sensorob_description/meshes/link_2_1.stl" scale="0.001 0.001 0.001"/>
+      <mesh filename="package://sensorob_description/meshes/link_2.stl" scale="0.001 0.001 0.001"/>
     </geometry>
     <material name="silver"/>
@@ -60,9 +60,9 @@
     <origin xyz="0.023626 0.041765 -0.187444" rpy="0 0 0"/>
     <geometry>
-      <mesh filename="package://sensorob_description/meshes/link_2_1.stl" scale="0.001 0.001 0.001"/>
+      <mesh filename="package://sensorob_description/meshes/link_2.stl" scale="0.001 0.001 0.001"/>
     </geometry>
   </collision>
 </link>
-<link name="link_3_1">
+<link name="link_3">
   <inertial>
     <origin xyz="0.03341663223535368 0.015743461072743326 0.13201293251123314" rpy="0 0 0"/>
@@ -73,5 +73,5 @@
     <origin xyz="-0.004978 0.028427 -0.612445" rpy="0 0 0"/>
     <geometry>
-      <mesh filename="package://sensorob_description/meshes/link_3_1.stl" scale="0.001 0.001 0.001"/>
+      <mesh filename="package://sensorob_description/meshes/link_3.stl" scale="0.001 0.001 0.001"/>
     </geometry>
     <material name="silver"/>
@@ -80,9 +80,9 @@
     <origin xyz="-0.004978 0.028427 -0.612445" rpy="0 0 0"/>
     <geometry>
-      <mesh filename="package://sensorob_description/meshes/link_3_1.stl" scale="0.001 0.001 0.001"/>
+      <mesh filename="package://sensorob_description/meshes/link_3.stl" scale="0.001 0.001 0.001"/>
     </geometry>
   </collision>
 </link>
-<link name="link_4_1">
+<link name="link_4">
   <inertial>
     <origin xyz="0.03362129286277545 0.015876430068886876 0.11081132606474609" rpy="0 0 0"/>
@@ -93,5 +93,5 @@
     <origin xyz="-0.038874 0.012621 -0.86107" rpy="0 0 0"/>
     <geometry>
-      <mesh filename="package://sensorob_description/meshes/link_4_1.stl" scale="0.001 0.001 0.001"/>
+      <mesh filename="package://sensorob_description/meshes/link_4.stl" scale="0.001 0.001 0.001"/>
     </geometry>
     <material name="silver"/>
@@ -100,18 +100,18 @@
     <origin xyz="-0.038874 0.012621 -0.86107" rpy="0 0 0"/>
     <geometry>
-      <mesh filename="package://sensorob_description/meshes/link_4_1.stl" scale="0.001 0.001 0.001"/>
+      <mesh filename="package://sensorob_description/meshes/link_4.stl" scale="0.001 0.001 0.001"/>
     </geometry>
   </collision>
 </link>
-<link name="link_5_1">
+<link name="link_5">
   <inertial>
-    <origin xyz="-0.01380891615594925 -0.00696923962437411 0.11701300634930023" rpy="0 0 0"/>
-    <mass value="1.1075042835385005"/>
-    <inertia ixx="0.005992" iyy="0.005957" izz="0.00149" ixy="3.4e-05" iyz="-0.000164" ixz="-0.000365"/>
+    <origin xyz="-0.013801299868957234 -0.00696463747478801 0.11721977365765945" rpy="0 0 0"/>
+    <mass value="1.10970553090912"/>
+    <inertia ixx="0.006017" iyy="0.005981" izz="0.001491" ixy="3.4e-05" iyz="-0.000165" ixz="-0.000366"/>
   </inertial>
   <visual>
     <origin xyz="-0.013787 0.024319 -1.004695" rpy="0 0 0"/>
     <geometry>
-      <mesh filename="package://sensorob_description/meshes/link_5_1.stl" scale="0.001 0.001 0.001"/>
+      <mesh filename="package://sensorob_description/meshes/link_5.stl" scale="0.001 0.001 0.001"/>
     </geometry>
     <material name="silver"/>
@@ -120,25 +120,25 @@
     <origin xyz="-0.013787 0.024319 -1.004695" rpy="0 0 0"/>
     <geometry>
-      <mesh filename="package://sensorob_description/meshes/link_5_1.stl" scale="0.001 0.001 0.001"/>
+      <mesh filename="package://sensorob_description/meshes/link_5.stl" scale="0.001 0.001 0.001"/>
     </geometry>
   </collision>
 </link>
-<link name="link_6_1">
+<link name="link_6">
   <inertial>
-    <origin xyz="-0.018743349594609954 0.024426822589732673 0.005589914717348821" rpy="0 0 0"/>
-    <mass value="0.05448899240176654"/>
-    <inertia ixx="1e-05" iyy="1e-05" izz="1.9e-05" ixy="-0.0" iyz="-0.0" ixz="0.0"/>
+    <origin xyz="-3.4959433121376643e-07 -1.774095831907907e-07 0.005353824436649113" rpy="0 0 0"/>
+    <mass value="0.04766984698965481"/>
+    <inertia ixx="9e-06" iyy="9e-06" izz="1.7e-05" ixy="0.0" iyz="-0.0" ixz="0.0"/>
   </inertial>
   <visual>
-    <origin xyz="-0.022561 0.053395 -1.225445" rpy="0 0 0"/>
+    <origin xyz="-0.003818 0.028968 -1.226445" rpy="0 0 0"/>
     <geometry>
-      <mesh filename="package://sensorob_description/meshes/link_6_1.stl" scale="0.001 0.001 0.001"/>
+      <mesh filename="package://sensorob_description/meshes/link_6.stl" scale="0.001 0.001 0.001"/>
     </geometry>
     <material name="silver"/>
   </visual>
   <collision>
-    <origin xyz="-0.022561 0.053395 -1.225445" rpy="0 0 0"/>
+    <origin xyz="-0.003818 0.028968 -1.226445" rpy="0 0 0"/>
     <geometry>
-      <mesh filename="package://sensorob_description/meshes/link_6_1.stl" scale="0.001 0.001 0.001"/>
+      <mesh filename="package://sensorob_description/meshes/link_6.stl" scale="0.001 0.001 0.001"/>
     </geometry>
   </collision>
@@ -147,5 +147,5 @@
   <origin xyz="0.06828 0.001091 0.070444" rpy="0 0 0"/>
   <parent link="base_link"/>
-  <child link="link_1_1"/>
+  <child link="link_1"/>
   <axis xyz="0.0 -0.0 1.0"/>
   <limit upper="2.181662" lower="-2.96706" effort="100" velocity="100"/>
@@ -153,6 +153,6 @@
 <joint name="joint_2" type="revolute">
   <origin xyz="-0.091906 -0.042856 0.117" rpy="0 0 0"/>
-  <parent link="link_1_1"/>
-  <child link="link_2_1"/>
+  <parent link="link_1"/>
+  <child link="link_2"/>
   <axis xyz="-0.906308 -0.422618 0.0"/>
   <limit upper="2.007129" lower="-2.007129" effort="100" velocity="100"/>
@@ -160,6 +160,6 @@
 <joint name="joint_3" type="revolute">
   <origin xyz="0.028604 0.013338 0.425001" rpy="0 0 0"/>
-  <parent link="link_2_1"/>
-  <child link="link_3_1"/>
+  <parent link="link_2"/>
+  <child link="link_3"/>
   <axis xyz="0.906308 0.422618 -0.0"/>
   <limit upper="2.879793" lower="-2.792527" effort="100" velocity="100"/>
@@ -167,19 +167,20 @@
 <joint name="joint_4" type="revolute">
   <origin xyz="0.033896 0.015806 0.248625" rpy="0 0 0"/>
-  <parent link="link_3_1"/>
-  <child link="link_4_1"/>
+  <parent link="link_3"/>
+  <child link="link_4"/>
   <axis xyz="0.0 0.0 1.0"/>
   <limit upper="4.45059" lower="-1.658063" effort="100" velocity="100"/>
 </joint>
-<joint name="joint_5" type="continuous">
+<joint name="joint_5" type="revolute">
   <origin xyz="-0.025087 -0.011698 0.143625" rpy="0 0 0"/>
-  <parent link="link_4_1"/>
-  <child link="link_5_1"/>
+  <parent link="link_4"/>
+  <child link="link_5"/>
   <axis xyz="-0.906308 -0.422618 -0.0"/>
+  <limit upper="2.96706" lower="-2.96706" effort="100" velocity="100"/>
 </joint>
 <joint name="joint_6" type="revolute">
-  <origin xyz="0.008774 -0.029076 0.22075" rpy="0 0 0"/>
-  <parent link="link_5_1"/>
-  <child link="link_6_1"/>
+  <origin xyz="-0.009969 -0.004649 0.22175" rpy="0 0 0"/>
+  <parent link="link_5"/>
+  <child link="link_6"/>
   <axis xyz="-0.0 -0.0 1.0"/>
   <limit upper="3.141593" lower="-3.141593" effort="100" velocity="100"/>
