Commit message: description

File: sensorob_description/urdf/materials.xacro (robot description, xacro)
@@ -1,6 +1,21 @@
 <?xml version="1.0" ?>
-<robot name="sensorob" xmlns:xacro="http://www.ros.org/wiki/xacro" >
-<material name="silver">
-  <color rgba="0.700 0.700 0.700 1.000"/>
-</material>
+<robot xmlns:xacro="http://www.ros.org/wiki/xacro" >
+    <material name="silver">
+        <color rgba="0.7 0.7 0.7 1"/>
+    </material>
+    <material name="white">
+        <color rgba="1 1 1 1" />
+    </material>
+    <material name="orange">
+        <color rgba="1 0.3 0.1 1"/>
+    </material>
+    <material name="blue">
+        <color rgba="0.2 0.2 1 1"/>
+    </material>
+    <material name="black">
+        <color rgba="0 0 0 1"/>
+    </material>
+    <material name="red">
+        <color rgba="1 0 0 1"/>
+    </material>
 </robot>
