Commit message: urdf edited

File: sensorob_description/urdf/robot_core.xacro (robot description, xacro)
@@ -14,5 +14,5 @@
       <origin xyz="0 0 0" rpy="0 0 0"/>
       <geometry>
-        <mesh filename="file://$(find sensorob_description)/meshes/base_link.stl" scale="0.001 0.001 0.001"/>
+       <mesh filename="file://$(find sensorob_description)/meshes/base_link.stl" scale="0.001 0.001 0.001"/>
       </geometry>
       <material name="white"/>
@@ -21,5 +21,5 @@
       <origin xyz="0 0 0" rpy="0 0 0"/>
       <geometry>
-        <mesh filename="file://$(find sensorob_description)/meshes/base_link.stl" scale="0.001 0.001 0.001"/>
+       <mesh filename="file://$(find sensorob_description)/meshes/base_link.stl" scale="0.001 0.001 0.001"/>
       </geometry>
     </collision>
@@ -27,12 +27,12 @@
   <link name="link_1">
     <inertial>
-      <origin xyz="-0.017391128474433415 -0.007793862548282313 0.09170345730211693" rpy="0 0 0"/>
+      <origin xyz="-0.019055565879578885 0.000286070591079963 0.09170345730211701" rpy="0 0 0"/>
       <mass value="2.1673778446055563"/>
-      <inertia ixx="0.006827" iyy="0.00695" izz="0.005681" ixy="-0.000182" iyz="0.00035" ixz="0.000778"/>
+      <inertia ixx="0.006709" iyy="0.007067" izz="0.005681" ixy="-7e-05" iyz="-1.2e-05" ixz="0.000853"/>
     </inertial>
     <visual>
       <origin xyz="-0.06828 -0.001091 -0.070444" rpy="0 0 0"/>
       <geometry>
-        <mesh filename="file://$(find sensorob_description)/meshes/link_1.stl" scale="0.001 0.001 0.001"/>
+       <mesh filename="file://$(find sensorob_description)/meshes/link_1.stl" scale="0.001 0.001 0.001"/>
       </geometry>
       <material name="white"/>
@@ -41,5 +41,5 @@
       <origin xyz="-0.06828 -0.001091 -0.070444" rpy="0 0 0"/>
       <geometry>
-        <mesh filename="file://$(find sensorob_description)/meshes/link_1.stl" scale="0.001 0.001 0.001"/>
+       <mesh filename="file://$(find sensorob_description)/meshes/link_1.stl" scale="0.001 0.001 0.001"/>
       </geometry>
     </collision>
@@ -47,19 +47,19 @@
   <link name="link_2">
     <inertial>
-      <origin xyz="-0.03597352078588314 -0.017962304231270702 0.2436907782754546" rpy="0 0 0"/>
+      <origin xyz="-0.04019415358244168 -0.0010759815082936714 0.2436907782754546" rpy="0 0 0"/>
       <mass value="3.7950516594171546"/>
-      <inertia ixx="0.123994" iyy="0.117506" izz="0.018463" ixy="0.003737" iyz="-0.000547" ixz="-0.00102"/>
+      <inertia ixx="0.125698" iyy="0.115802" izz="0.018463" ixy="-8.3e-05" iyz="-6.5e-05" ixz="-0.001156"/>
     </inertial>
     <visual>
-      <origin xyz="0.023626 0.041765 -0.187444" rpy="0 0 0"/>
+      <origin xyz="0.033127 -0.001091 -0.187444" rpy="0 0 0"/>
       <geometry>
-        <mesh filename="file://$(find sensorob_description)/meshes/link_2.stl" scale="0.001 0.001 0.001"/>
+       <mesh filename="file://$(find sensorob_description)/meshes/link_2.stl" scale="0.001 0.001 0.001"/>
       </geometry>
       <material name="white"/>
     </visual>
     <collision>
-      <origin xyz="0.023626 0.041765 -0.187444" rpy="0 0 0"/>
+      <origin xyz="0.033127 -0.001091 -0.187444" rpy="0 0 0"/>
       <geometry>
-        <mesh filename="file://$(find sensorob_description)/meshes/link_2.stl" scale="0.001 0.001 0.001"/>
+       <mesh filename="file://$(find sensorob_description)/meshes/link_2.stl" scale="0.001 0.001 0.001"/>
       </geometry>
     </collision>
@@ -67,19 +67,19 @@
   <link name="link_3">
     <inertial>
-      <origin xyz="0.03341663223535368 0.015743461072743326 0.13201293251123314" rpy="0 0 0"/>
+      <origin xyz="0.03693926470328392 0.0001460307076859913 0.13201293251123314" rpy="0 0 0"/>
       <mass value="1.1351525716942115"/>
-      <inertia ixx="0.007184" iyy="0.007038" izz="0.001398" ixy="9.8e-05" iyz="-2.7e-05" ixz="-7.1e-05"/>
+      <inertia ixx="0.007232" iyy="0.006989" izz="0.001398" ixy="7e-06" iyz="6e-06" ixz="-7.5e-05"/>
     </inertial>
     <visual>
-      <origin xyz="-0.004978 0.028427 -0.612445" rpy="0 0 0"/>
+      <origin xyz="0.001566 -0.001091 -0.612445" rpy="0 0 0"/>
       <geometry>
-        <mesh filename="file://$(find sensorob_description)/meshes/link_3.stl" scale="0.001 0.001 0.001"/>
+       <mesh filename="file://$(find sensorob_description)/meshes/link_3.stl" scale="0.001 0.001 0.001"/>
       </geometry>
       <material name="white"/>
     </visual>
     <collision>
-      <origin xyz="-0.004978 0.028427 -0.612445" rpy="0 0 0"/>
+      <origin xyz="0.001566 -0.001091 -0.612445" rpy="0 0 0"/>
       <geometry>
-        <mesh filename="file://$(find sensorob_description)/meshes/link_3.stl" scale="0.001 0.001 0.001"/>
+       <mesh filename="file://$(find sensorob_description)/meshes/link_3.stl" scale="0.001 0.001 0.001"/>
       </geometry>
     </collision>
@@ -87,19 +87,19 @@
   <link name="link_4">
     <inertial>
-      <origin xyz="0.03362129286277545 0.015876430068886876 0.11081132606474609" rpy="0 0 0"/>
+      <origin xyz="0.03718105834409844 0.00018008050762574395 0.11081132606474409" rpy="0 0 0"/>
       <mass value="1.2025016995467235"/>
-      <inertia ixx="0.004179" iyy="0.004517" izz="0.002169" ixy="-0.000203" iyz="-0.000281" ixz="-0.000573"/>
+      <inertia ixx="0.004084" iyy="0.004612" izz="0.002169" ixy="-1e-06" iyz="-1.3e-05" ixz="-0.000638"/>
     </inertial>
     <visual>
-      <origin xyz="-0.038874 0.012621 -0.86107" rpy="0 0 0"/>
+      <origin xyz="-0.035834 -0.001091 -0.86107" rpy="0 0 0"/>
       <geometry>
-        <mesh filename="file://$(find sensorob_description)/meshes/link_4.stl" scale="0.001 0.001 0.001"/>
+       <mesh filename="file://$(find sensorob_description)/meshes/link_4.stl" scale="0.001 0.001 0.001"/>
       </geometry>
       <material name="white"/>
     </visual>
     <collision>
-      <origin xyz="-0.038874 0.012621 -0.86107" rpy="0 0 0"/>
+      <origin xyz="-0.035834 -0.001091 -0.86107" rpy="0 0 0"/>
       <geometry>
-        <mesh filename="file://$(find sensorob_description)/meshes/link_4.stl" scale="0.001 0.001 0.001"/>
+       <mesh filename="file://$(find sensorob_description)/meshes/link_4.stl" scale="0.001 0.001 0.001"/>
       </geometry>
     </collision>
@@ -107,19 +107,19 @@
   <link name="link_5">
     <inertial>
-      <origin xyz="-0.013801299868957234 -0.00696463747478801 0.11721977365765945" rpy="0 0 0"/>
+      <origin xyz="-0.01545179087098288 -0.0004790673243868698 0.11721977365765723" rpy="0 0 0"/>
       <mass value="1.10970553090912"/>
-      <inertia ixx="0.006017" iyy="0.005981" izz="0.001491" ixy="3.4e-05" iyz="-0.000165" ixz="-0.000366"/>
+      <inertia ixx="0.006037" iyy="0.005961" izz="0.001491" ixy="9e-06" iyz="5e-06" ixz="-0.000401"/>
     </inertial>
     <visual>
-      <origin xyz="-0.013787 0.024319 -1.004695" rpy="0 0 0"/>
+      <origin xyz="-0.008154 -0.001091 -1.004695" rpy="0 0 0"/>
       <geometry>
-        <mesh filename="file://$(find sensorob_description)/meshes/link_5.stl" scale="0.001 0.001 0.001"/>
+       <mesh filename="file://$(find sensorob_description)/meshes/link_5.stl" scale="0.001 0.001 0.001"/>
       </geometry>
       <material name="white"/>
     </visual>
     <collision>
-      <origin xyz="-0.013787 0.024319 -1.004695" rpy="0 0 0"/>
+      <origin xyz="-0.008154 -0.001091 -1.004695" rpy="0 0 0"/>
       <geometry>
-        <mesh filename="file://$(find sensorob_description)/meshes/link_5.stl" scale="0.001 0.001 0.001"/>
+       <mesh filename="file://$(find sensorob_description)/meshes/link_5.stl" scale="0.001 0.001 0.001"/>
       </geometry>
     </collision>
@@ -127,19 +127,19 @@
   <link name="link_6">
     <inertial>
-      <origin xyz="-3.4959433121376643e-07 -1.774095831907907e-07 0.005353824436649113" rpy="0 0 0"/>
+      <origin xyz="-3.087896676863544e-07 -8.620905638662135e-13 0.005353824436647114" rpy="0 0 0"/>
       <mass value="0.04766984698965481"/>
-      <inertia ixx="9e-06" iyy="9e-06" izz="1.7e-05" ixy="0.0" iyz="-0.0" ixz="0.0"/>
+      <inertia ixx="9e-06" iyy="9e-06" izz="1.7e-05" ixy="-0.0" iyz="-0.0" ixz="0.0"/>
     </inertial>
     <visual>
-      <origin xyz="-0.003818 0.028968 -1.226445" rpy="0 0 0"/>
+      <origin xyz="0.002846 -0.001091 -1.226445" rpy="0 0 0"/>
       <geometry>
-        <mesh filename="file://$(find sensorob_description)/meshes/link_6.stl" scale="0.001 0.001 0.001"/>
+       <mesh filename="file://$(find sensorob_description)/meshes/link_6.stl" scale="0.001 0.001 0.001"/>
       </geometry>
       <material name="white"/>
     </visual>
     <collision>
-      <origin xyz="-0.003818 0.028968 -1.226445" rpy="0 0 0"/>
+      <origin xyz="0.002846 -0.001091 -1.226445" rpy="0 0 0"/>
       <geometry>
-        <mesh filename="file://$(find sensorob_description)/meshes/link_6.stl" scale="0.001 0.001 0.001"/>
+       <mesh filename="file://$(find sensorob_description)/meshes/link_6.stl" scale="0.001 0.001 0.001"/>
       </geometry>
     </collision>
@@ -154,42 +154,41 @@
     <parent link="base_link"/>
     <child link="link_1"/>
-    <axis xyz="0.0 -0.0 1.0"/>
-    <limit upper="2.181662" lower="-2.96706" effort="5" velocity="2"/>
-  <!--   <dynamics damping="100" friction="100"/>-->
+    <axis xyz="0.0 0.0 1.0"/>
+    <limit upper="2.181662" lower="-2.96706" effort="100" velocity="100"/>
   </joint>
   <joint name="joint_2" type="revolute">
-    <origin xyz="-0.091906 -0.042856 0.117" rpy="0 0 0"/>
+    <origin xyz="-0.101407 0.0 0.117" rpy="0 0 0"/>
     <parent link="link_1"/>
     <child link="link_2"/>
-    <axis xyz="-0.906308 -0.422618 0.0"/>
-    <limit upper="2.007129" lower="-2.007129" effort="5" velocity="2"/>
+    <axis xyz="-1.0 -0.0 0.0"/>
+    <limit upper="2.007129" lower="-2.007129" effort="100" velocity="100"/>
   </joint>
   <joint name="joint_3" type="revolute">
-    <origin xyz="0.028604 0.013338 0.425001" rpy="0 0 0"/>
+    <origin xyz="0.031561 0.0 0.425001" rpy="0 0 0"/>
     <parent link="link_2"/>
     <child link="link_3"/>
-    <axis xyz="0.906308 0.422618 -0.0"/>
-    <limit upper="2.879793" lower="-2.792527" effort="5" velocity="2"/>
+    <axis xyz="1.0 0.0 -0.0"/>
+    <limit upper="2.879793" lower="-2.792527" effort="100" velocity="100"/>
   </joint>
   <joint name="joint_4" type="revolute">
-    <origin xyz="0.033896 0.015806 0.248625" rpy="0 0 0"/>
+    <origin xyz="0.0374 0.0 0.248625" rpy="0 0 0"/>
     <parent link="link_3"/>
     <child link="link_4"/>
     <axis xyz="0.0 0.0 1.0"/>
-    <limit upper="4.45059" lower="-1.658063" effort="5" velocity="2"/>
+    <limit upper="4.45059" lower="-1.658063" effort="100" velocity="100"/>
   </joint>
   <joint name="joint_5" type="revolute">
-    <origin xyz="-0.025087 -0.011698 0.143625" rpy="0 0 0"/>
+    <origin xyz="-0.02768 0.0 0.143625" rpy="0 0 0"/>
     <parent link="link_4"/>
     <child link="link_5"/>
-    <axis xyz="-0.906308 -0.422618 -0.0"/>
-    <limit upper="2.96706" lower="-2.96706" effort="5" velocity="2"/>
+    <axis xyz="-1.0 -0.0 -0.0"/>
+    <limit upper="2.96706" lower="-2.96706" effort="100" velocity="100"/>
   </joint>
   <joint name="joint_6" type="revolute">
-    <origin xyz="-0.009969 -0.004649 0.22175" rpy="0 0 0"/>
+    <origin xyz="-0.011 0.0 0.22175" rpy="0 0 0"/>
     <parent link="link_5"/>
     <child link="link_6"/>
-    <axis xyz="-0.0 -0.0 1.0"/>
-    <limit upper="3.141593" lower="-3.141593" effort="5" velocity="2"/>
+    <axis xyz="-0.0 0.0 1.0"/>
+    <limit upper="3.141593" lower="-3.141593" effort="100" velocity="100"/>
   </joint>
 </robot>

File: sensorob_description/urdf/sensorob.urdf (robot description, URDF)
Before this commit: robot sensorob, 7 links, 6 joints
Links:
- added link world
- link base_link: geometry collision mesh filename=file:///home/jakub/ros2_ws/install/sensorob_description/sha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 scale=0.001 0.001 0.001; visual mesh filename=file:///home/jakub/ros2_ws/install/sensorob_description/sha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 scale=0.001 0.001 0.001
- link link_1: geometry collision mesh filename=file:///home/jakub/ros2_ws/install/sensorob_description/sha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 scale=0.001 0.001 0.001; visual mesh filename=file:///home/jakub/ros2_ws/install/sensorob_description/sha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 scale=0.001 0.001 0.001
- link link_2: geometry collision mesh filename=file:///home/jakub/ros2_ws/install/sensorob_description/sha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 scale=0.001 0.001 0.001; visual mesh filename=file:///home/jakub/ros2_ws/install/sensorob_description/sha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 scale=0.001 0.001 0.001
- link link_3: geometry collision mesh filename=file:///home/jakub/ros2_ws/install/sensorob_description/sha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 scale=0.001 0.001 0.001; visual mesh filename=file:///home/jakub/ros2_ws/install/sensorob_description/sha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 scale=0.001 0.001 0.001
- link link_4: geometry collision mesh filename=file:///home/jakub/ros2_ws/install/sensorob_description/sha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 scale=0.001 0.001 0.001; visual mesh filename=file:///home/jakub/ros2_ws/install/sensorob_description/sha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 scale=0.001 0.001 0.001
- link link_5: geometry collision mesh filename=file:///home/jakub/ros2_ws/install/sensorob_description/sha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 scale=0.001 0.001 0.001; visual mesh filename=file:///home/jakub/ros2_ws/install/sensorob_description/sha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 scale=0.001 0.001 0.001
- link link_6: geometry collision mesh filename=file:///home/jakub/ros2_ws/install/sensorob_description/sha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 scale=0.001 0.001 0.001; visual mesh filename=file:///home/jakub/ros2_ws/install/sensorob_description/sha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 scale=0.001 0.001 0.001
Joints:
- added joint world_link_joint: type fixed, parent world, child base_link, origin xyz=0.05 0.05 0.2 rpy=0 0 0
- joint joint_1: axis 0.0 -0.0 1.0 -> 0.0 0.0 1.0
- joint joint_2: axis -0.906308 -0.422618 0.0 -> -1.0 -0.0 0.0; origin xyz=-0.091906 -0.042856 0.117 rpy=0 0 0 -> xyz=-0.101407 0.0 0.117 rpy=0 0 0
- joint joint_3: axis 0.906308 0.422618 -0.0 -> 1.0 0.0 -0.0; origin xyz=0.028604 0.013338 0.425001 rpy=0 0 0 -> xyz=0.031561 0.0 0.425001 rpy=0 0 0
- joint joint_4: origin xyz=0.033896 0.015806 0.248625 rpy=0 0 0 -> xyz=0.0374 0.0 0.248625 rpy=0 0 0
- joint joint_5: axis -0.906308 -0.422618 -0.0 -> -1.0 -0.0 -0.0; origin xyz=-0.025087 -0.011698 0.143625 rpy=0 0 0 -> xyz=-0.02768 0.0 0.143625 rpy=0 0 0
- joint joint_6: axis -0.0 -0.0 1.0 -> -0.0 0.0 1.0; origin xyz=-0.009969 -0.004649 0.22175 rpy=0 0 0 -> xyz=-0.011 0.0 0.22175 rpy=0 0 0

Commit message: model edit

File: sensorob_description/urdf/robot_core.xacro (robot description, xacro)
@@ -127,19 +127,19 @@
   <link name="link_6">
     <inertial>
-      <origin xyz="-3.087896676863544e-07 -8.620905638662135e-13 0.005353824436647114" rpy="0 0 0"/>
+      <origin xyz="-3.0879003850084463e-07 9.529287081644355e-13 0.005353824436650445" rpy="0 0 0"/>
       <mass value="0.04766984698965481"/>
-      <inertia ixx="9e-06" iyy="9e-06" izz="1.7e-05" ixy="-0.0" iyz="-0.0" ixz="0.0"/>
+      <inertia ixx="9e-06" iyy="9e-06" izz="1.7e-05" ixy="-0.0" iyz="0.0" ixz="-0.0"/>
     </inertial>
     <visual>
       <origin xyz="0.002846 -0.001091 -1.226445" rpy="0 0 0"/>
       <geometry>
-       <mesh filename="file://$(find sensorob_description)/meshes/link_6.stl" scale="0.001 0.001 0.001"/>
+        <mesh filename="file://$(find sensorob_description)/meshes/link_6.stl" scale="0.001 0.001 0.001"/>
       </geometry>
-      <material name="white"/>
+      <material name="silver"/>
     </visual>
     <collision>
       <origin xyz="0.002846 -0.001091 -1.226445" rpy="0 0 0"/>
       <geometry>
-       <mesh filename="file://$(find sensorob_description)/meshes/link_6.stl" scale="0.001 0.001 0.001"/>
+        <mesh filename="file://$(find sensorob_description)/meshes/link_6.stl" scale="0.001 0.001 0.001"/>
       </geometry>
     </collision>

Commit message: model edit v2 + kinematics config

File: sensorob_description/urdf/robot_core.xacro (robot description, xacro)
@@ -7,5 +7,5 @@
   <link name="base_link">
     <inertial>
-      <origin xyz="0.06842933950869011 0.0009438578686686358 -0.026799613448182" rpy="0 0 0"/>
+      <origin xyz="0.0684293395086911 0.0009438578686822592 -0.026799613448182283" rpy="0 0 0"/>
       <mass value="1.855542034998811"/>
       <inertia ixx="0.00951" iyy="0.008318" izz="0.007035" ixy="1e-05" iyz="-2.2e-05" ixz="2.3e-05"/>
@@ -27,5 +27,5 @@
   <link name="link_1">
     <inertial>
-      <origin xyz="-0.019055565879578885 0.000286070591079963 0.09170345730211701" rpy="0 0 0"/>
+      <origin xyz="-0.019055565879577983 0.00028607059109358383 0.0917034573021166" rpy="0 0 0"/>
       <mass value="2.1673778446055563"/>
       <inertia ixx="0.006709" iyy="0.007067" izz="0.005681" ixy="-7e-05" iyz="-1.2e-05" ixz="0.000853"/>
@@ -47,5 +47,5 @@
   <link name="link_2">
     <inertial>
-      <origin xyz="-0.04019415358244168 -0.0010759815082936714 0.2436907782754546" rpy="0 0 0"/>
+      <origin xyz="-0.04019415358244136 -0.0010759815082800456 0.24369077827545405" rpy="0 0 0"/>
       <mass value="3.7950516594171546"/>
       <inertia ixx="0.125698" iyy="0.115802" izz="0.018463" ixy="-8.3e-05" iyz="-6.5e-05" ixz="-0.001156"/>
@@ -87,5 +87,5 @@
   <link name="link_4">
     <inertial>
-      <origin xyz="0.03718105834409844 0.00018008050762574395 0.11081132606474409" rpy="0 0 0"/>
+      <origin xyz="0.037181058344095096 0.0001800805076532456 0.11081132606474708" rpy="0 0 0"/>
       <mass value="1.2025016995467235"/>
       <inertia ixx="0.004084" iyy="0.004612" izz="0.002169" ixy="-1e-06" iyz="-1.3e-05" ixz="-0.000638"/>
@@ -107,5 +107,5 @@
   <link name="link_5">
     <inertial>
-      <origin xyz="-0.01545179087098288 -0.0004790673243868698 0.11721977365765723" rpy="0 0 0"/>
+      <origin xyz="-0.015451790870986186 -0.0004790673243593754 0.11721977365766034" rpy="0 0 0"/>
       <mass value="1.10970553090912"/>
       <inertia ixx="0.006037" iyy="0.005961" izz="0.001491" ixy="9e-06" iyz="5e-06" ixz="-0.000401"/>
@@ -114,5 +114,5 @@
       <origin xyz="-0.008154 -0.001091 -1.004695" rpy="0 0 0"/>
       <geometry>
-       <mesh filename="file://$(find sensorob_description)/meshes/link_5.stl" scale="0.001 0.001 0.001"/>
+        <mesh filename="file://$(find sensorob_description)/meshes/link_5.stl" scale="0.001 0.001 0.001"/>
       </geometry>
       <material name="white"/>
@@ -121,5 +121,5 @@
       <origin xyz="-0.008154 -0.001091 -1.004695" rpy="0 0 0"/>
       <geometry>
-       <mesh filename="file://$(find sensorob_description)/meshes/link_5.stl" scale="0.001 0.001 0.001"/>
+        <mesh filename="file://$(find sensorob_description)/meshes/link_5.stl" scale="0.001 0.001 0.001"/>
       </geometry>
     </collision>
@@ -127,7 +127,7 @@
   <link name="link_6">
     <inertial>
-      <origin xyz="-3.0879003850084463e-07 9.529287081644355e-13 0.005353824436650445" rpy="0 0 0"/>
+      <origin xyz="-3.0878998574747005e-07 -8.994784084226382e-13 0.005353824436650445" rpy="0 0 0"/>
       <mass value="0.04766984698965481"/>
-      <inertia ixx="9e-06" iyy="9e-06" izz="1.7e-05" ixy="-0.0" iyz="0.0" ixz="-0.0"/>
+      <inertia ixx="9e-06" iyy="9e-06" izz="1.7e-05" ixy="-0.0" iyz="-0.0" ixz="0.0"/>
     </inertial>
     <visual>
@@ -136,5 +136,5 @@
         <mesh filename="file://$(find sensorob_description)/meshes/link_6.stl" scale="0.001 0.001 0.001"/>
       </geometry>
-      <material name="silver"/>
+      <material name="white"/>
     </visual>
     <collision>
@@ -154,5 +154,5 @@
     <parent link="base_link"/>
     <child link="link_1"/>
-    <axis xyz="0.0 0.0 1.0"/>
+    <axis xyz="0.0 -0.0 1.0"/>
     <limit upper="2.181662" lower="-2.96706" effort="100" velocity="100"/>
   </joint>
@@ -161,5 +161,5 @@
     <parent link="link_1"/>
     <child link="link_2"/>
-    <axis xyz="-1.0 -0.0 0.0"/>
+    <axis xyz="-1.0 0.0 -0.0"/>
     <limit upper="2.007129" lower="-2.007129" effort="100" velocity="100"/>
   </joint>
@@ -168,5 +168,5 @@
     <parent link="link_2"/>
     <child link="link_3"/>
-    <axis xyz="1.0 0.0 -0.0"/>
+    <axis xyz="1.0 0.0 0.0"/>
     <limit upper="2.879793" lower="-2.792527" effort="100" velocity="100"/>
   </joint>
@@ -182,5 +182,5 @@
     <parent link="link_4"/>
     <child link="link_5"/>
-    <axis xyz="-1.0 -0.0 -0.0"/>
+    <axis xyz="-1.0 -0.0 0.0"/>
     <limit upper="2.96706" lower="-2.96706" effort="100" velocity="100"/>
   </joint>
@@ -189,6 +189,6 @@
     <parent link="link_5"/>
     <child link="link_6"/>
-    <axis xyz="-0.0 0.0 1.0"/>
-    <limit upper="3.141593" lower="-3.141593" effort="100" velocity="100"/>
+    <axis xyz="0.0 -0.0 -1.0"/>
+    <limit upper="2.792527" lower="-2.792527" effort="100" velocity="100"/>
   </joint>
 </robot>

File: sensorob_description/urdf/sensorob.urdf (robot description, URDF)
Before this commit: robot sensorob, 8 links, 7 joints
Joints:
- joint joint_1: axis 0.0 0.0 1.0 -> 0.0 -0.0 1.0
- joint joint_2: axis -1.0 -0.0 0.0 -> -1.0 0.0 -0.0
- joint joint_3: axis 1.0 0.0 -0.0 -> 1.0 0.0 0.0
- joint joint_5: axis -1.0 -0.0 -0.0 -> -1.0 -0.0 0.0
- joint joint_6: axis -0.0 0.0 1.0 -> 0.0 -0.0 -1.0; limit lower=-3.141593 upper=3.141593 effort=100 velocity=100 -> lower=-2.792527 upper=2.792527 effort=100 velocity=100

File: sensorob_moveit_config/config/sensorob.urdf.xacro (robot description, xacro)
@@ -1,9 +1,5 @@
-<?xml version="1.0"?>
-<robot xmlns:xacro="http://www.ros.org/wiki/xacro" name="sensorob">
-    <xacro:arg name="initial_positions_file" default="initial_positions.yaml" />
-    <!-- Import sensorob urdf file -->
-    <xacro:include filename="$(find sensorob_description)/urdf/sensorob.urdf.xacro" />
-    <!-- Import control_xacro -->
-    <xacro:include filename="sensorob.ros2_control.xacro" />
-    <xacro:sensorob_ros2_control name="FakeSystem" initial_positions_file="$(arg initial_positions_file)"/>
+<?xml version="1.0" ?>
+<robot name="sensorob" xmlns:xacro="http://www.ros.org/wiki/xacro">
+  <xacro:include filename="robot_core.xacro" />
+  <xacro:include filename="$(find sensorob_description)/urdf/ros2_control.xacro" />
 </robot>
