Commit message: description and config package

File: sensorob_description/urdf/robot_core.xacro (robot description, xacro)
@@ -14,5 +14,5 @@
       <origin xyz="0 0 0" rpy="0 0 0"/>
       <geometry>
-       <mesh filename="file://$(find sensorob_description)/meshes/base_link.stl" scale="0.001 0.001 0.001"/>
+        <mesh filename="file://$(find sensorob_description)/meshes/base_link.stl" scale="0.001 0.001 0.001"/>
       </geometry>
       <material name="white"/>
@@ -21,5 +21,5 @@
       <origin xyz="0 0 0" rpy="0 0 0"/>
       <geometry>
-       <mesh filename="file://$(find sensorob_description)/meshes/base_link.stl" scale="0.001 0.001 0.001"/>
+        <mesh filename="file://$(find sensorob_description)/meshes/base_link.stl" scale="0.001 0.001 0.001"/>
       </geometry>
     </collision>
@@ -34,5 +34,5 @@
       <origin xyz="-0.06828 -0.001091 -0.070444" rpy="0 0 0"/>
       <geometry>
-       <mesh filename="file://$(find sensorob_description)/meshes/link_1.stl" scale="0.001 0.001 0.001"/>
+        <mesh filename="file://$(find sensorob_description)/meshes/link_1.stl" scale="0.001 0.001 0.001"/>
       </geometry>
       <material name="white"/>
@@ -41,5 +41,5 @@
       <origin xyz="-0.06828 -0.001091 -0.070444" rpy="0 0 0"/>
       <geometry>
-       <mesh filename="file://$(find sensorob_description)/meshes/link_1.stl" scale="0.001 0.001 0.001"/>
+        <mesh filename="file://$(find sensorob_description)/meshes/link_1.stl" scale="0.001 0.001 0.001"/>
       </geometry>
     </collision>
@@ -54,5 +54,5 @@
       <origin xyz="0.033127 -0.001091 -0.187444" rpy="0 0 0"/>
       <geometry>
-       <mesh filename="file://$(find sensorob_description)/meshes/link_2.stl" scale="0.001 0.001 0.001"/>
+        <mesh filename="file://$(find sensorob_description)/meshes/link_2.stl" scale="0.001 0.001 0.001"/>
       </geometry>
       <material name="white"/>
@@ -61,5 +61,5 @@
       <origin xyz="0.033127 -0.001091 -0.187444" rpy="0 0 0"/>
       <geometry>
-       <mesh filename="file://$(find sensorob_description)/meshes/link_2.stl" scale="0.001 0.001 0.001"/>
+        <mesh filename="file://$(find sensorob_description)/meshes/link_2.stl" scale="0.001 0.001 0.001"/>
       </geometry>
     </collision>
@@ -74,5 +74,5 @@
       <origin xyz="0.001566 -0.001091 -0.612445" rpy="0 0 0"/>
       <geometry>
-       <mesh filename="file://$(find sensorob_description)/meshes/link_3.stl" scale="0.001 0.001 0.001"/>
+        <mesh filename="file://$(find sensorob_description)/meshes/link_3.stl" scale="0.001 0.001 0.001"/>
       </geometry>
       <material name="white"/>
@@ -81,5 +81,5 @@
       <origin xyz="0.001566 -0.001091 -0.612445" rpy="0 0 0"/>
       <geometry>
-       <mesh filename="file://$(find sensorob_description)/meshes/link_3.stl" scale="0.001 0.001 0.001"/>
+        <mesh filename="file://$(find sensorob_description)/meshes/link_3.stl" scale="0.001 0.001 0.001"/>
       </geometry>
     </collision>
@@ -94,5 +94,5 @@
       <origin xyz="-0.035834 -0.001091 -0.86107" rpy="0 0 0"/>
       <geometry>
-       <mesh filename="file://$(find sensorob_description)/meshes/link_4.stl" scale="0.001 0.001 0.001"/>
+        <mesh filename="file://$(find sensorob_description)/meshes/link_4.stl" scale="0.001 0.001 0.001"/>
       </geometry>
       <material name="white"/>
@@ -101,5 +101,5 @@
       <origin xyz="-0.035834 -0.001091 -0.86107" rpy="0 0 0"/>
       <geometry>
-       <mesh filename="file://$(find sensorob_description)/meshes/link_4.stl" scale="0.001 0.001 0.001"/>
+        <mesh filename="file://$(find sensorob_description)/meshes/link_4.stl" scale="0.001 0.001 0.001"/>
       </geometry>
     </collision>
@@ -155,5 +155,5 @@
     <child link="link_1"/>
     <axis xyz="0.0 -0.0 1.0"/>
-    <limit upper="2.181662" lower="-2.96706" effort="100" velocity="100"/>
+    <limit upper="3.141592653589793" lower="-3.141592653589793" effort="100" velocity="100"/> <!-- +-pi -->
   </joint>
   <joint name="joint_2" type="revolute">
@@ -162,5 +162,5 @@
     <child link="link_2"/>
     <axis xyz="-1.0 0.0 -0.0"/>
-    <limit upper="2.007129" lower="-2.007129" effort="100" velocity="100"/>
+    <limit upper="1.570796327" lower="-1.570796327" effort="100" velocity="100"/> <!-- +-pi/2 -->
   </joint>
   <joint name="joint_3" type="revolute">
@@ -169,5 +169,5 @@
     <child link="link_3"/>
     <axis xyz="1.0 0.0 0.0"/>
-    <limit upper="2.879793" lower="-2.792527" effort="100" velocity="100"/>
+    <limit upper="2.094395102" lower="-2.094395102" effort="100" velocity="100"/> <!-- +-2pi/3-->
   </joint>
   <joint name="joint_4" type="revolute">
@@ -176,5 +176,5 @@
     <child link="link_4"/>
     <axis xyz="0.0 0.0 1.0"/>
-    <limit upper="4.45059" lower="-1.658063" effort="100" velocity="100"/>
+    <limit upper="3.141592653589793" lower="-3.141592653589793" effort="100" velocity="100"/> <!-- +-pi -->
   </joint>
   <joint name="joint_5" type="revolute">
@@ -183,5 +183,5 @@
     <child link="link_5"/>
     <axis xyz="-1.0 -0.0 0.0"/>
-    <limit upper="2.96706" lower="-2.96706" effort="100" velocity="100"/>
+    <limit upper="1.570796327" lower="-1.570796327" effort="100" velocity="100"/> <!-- +-pi/2 -->
   </joint>
   <joint name="joint_6" type="revolute">
@@ -190,5 +190,5 @@
     <child link="link_6"/>
     <axis xyz="0.0 -0.0 -1.0"/>
-    <limit upper="2.792527" lower="-2.792527" effort="100" velocity="100"/>
+    <limit upper="6.283185307" lower="-6.283185307" effort="100" velocity="100"/> <!-- +-2pi -->
   </joint>
 </robot>

File: sensorob_description/urdf/sensorob.urdf (robot description, URDF)
Before this commit: robot sensorob, 8 links, 7 joints
Joints:
- joint joint_1: limit lower=-2.96706 upper=2.181662 effort=100 velocity=100 -> lower=-3.141592653589793 upper=3.141592653589793 effort=100 velocity=100
- joint joint_2: limit lower=-2.007129 upper=2.007129 effort=100 velocity=100 -> lower=-1.570796327 upper=1.570796327 effort=100 velocity=100
- joint joint_3: limit lower=-2.792527 upper=2.879793 effort=100 velocity=100 -> lower=-2.094395102 upper=2.094395102 effort=100 velocity=100
- joint joint_4: limit lower=-1.658063 upper=4.45059 effort=100 velocity=100 -> lower=-3.141592653589793 upper=3.141592653589793 effort=100 velocity=100
- joint joint_5: limit lower=-2.96706 upper=2.96706 effort=100 velocity=100 -> lower=-1.570796327 upper=1.570796327 effort=100 velocity=100
- joint joint_6: limit lower=-2.792527 upper=2.792527 effort=100 velocity=100 -> lower=-6.283185307 upper=6.283185307 effort=100 velocity=100

Commit message: ros2_control + real hw implementation

File: sensorob_description/urdf/robot_core.xacro (robot description, xacro)
@@ -155,5 +155,5 @@
     <child link="link_1"/>
     <axis xyz="0.0 -0.0 1.0"/>
-    <limit upper="3.141592653589793" lower="-3.141592653589793" effort="100" velocity="100"/> <!-- +-pi -->
+    <limit upper="3.141592653589793" lower="-3.141592653589793" effort="500" velocity="6"/> <!-- +-pi -->
   </joint>
   <joint name="joint_2" type="revolute">
@@ -162,5 +162,5 @@
     <child link="link_2"/>
     <axis xyz="-1.0 0.0 -0.0"/>
-    <limit upper="1.570796327" lower="-1.570796327" effort="100" velocity="100"/> <!-- +-pi/2 -->
+    <limit upper="1.570796327" lower="-1.570796327" effort="500" velocity="6"/> <!-- +-pi/2 -->
   </joint>
   <joint name="joint_3" type="revolute">
@@ -169,5 +169,5 @@
     <child link="link_3"/>
     <axis xyz="1.0 0.0 0.0"/>
-    <limit upper="2.094395102" lower="-2.094395102" effort="100" velocity="100"/> <!-- +-2pi/3-->
+    <limit upper="2.094395102" lower="-2.094395102" effort="300" velocity="7"/> <!-- +-2pi/3-->
   </joint>
   <joint name="joint_4" type="revolute">
@@ -176,5 +176,5 @@
     <child link="link_4"/>
     <axis xyz="0.0 0.0 1.0"/>
-    <limit upper="3.141592653589793" lower="-3.141592653589793" effort="100" velocity="100"/> <!-- +-pi -->
+    <limit upper="3.141592653589793" lower="-3.141592653589793" effort="200" velocity="8"/> <!-- +-pi -->
   </joint>
   <joint name="joint_5" type="revolute">
@@ -183,5 +183,5 @@
     <child link="link_5"/>
     <axis xyz="-1.0 -0.0 0.0"/>
-    <limit upper="1.570796327" lower="-1.570796327" effort="100" velocity="100"/> <!-- +-pi/2 -->
+    <limit upper="1.570796327" lower="-1.570796327" effort="200" velocity="8"/> <!-- +-pi/2 -->
   </joint>
   <joint name="joint_6" type="revolute">
@@ -190,5 +190,5 @@
     <child link="link_6"/>
     <axis xyz="0.0 -0.0 -1.0"/>
-    <limit upper="6.283185307" lower="-6.283185307" effort="100" velocity="100"/> <!-- +-2pi -->
+    <limit upper="3.141592653589793" lower="-3.141592653589793" effort="200" velocity="10"/> <!-- +-pi (cannot be higher because of an absolut encoder without flash disk)-->
   </joint>
 </robot>

File: sensorob_description/urdf/ros2_control.xacro (robot description, xacro)
@@ -3,57 +3,4 @@
     <xacro:if value="$(arg sim_mode)">
         <ros2_control name="GazeboSystem" type="system">
-            <hardware>
-                <plugin>gazebo_ros2_control/GazeboSystem</plugin>
-            </hardware>
-            <joint name="joint_1">
-                <command_interface name="position"/>
-                <command_interface name="effort"/>
-    <!--            <command_interface name="velocity"/>-->
-    <!--            <command_interface name="effort"/>-->
-    <!--                <param name="min">-10</param>-->
-    <!--                <param name="max">10</param>-->
-                <state_interface name="position"/>
-                <state_interface name="velocity"/>
-                <state_interface name="effort"/>
-            </joint>
-            <joint name="joint_2">
-                <command_interface name="position"/>
-                <command_interface name="effort"/>
-                <state_interface name="position"/>
-                <state_interface name="velocity"/>
-                <state_interface name="effort"/>
-            </joint>
-            <joint name="joint_3">
-                <command_interface name="position"/>
-                <command_interface name="effort"/>
-                <state_interface name="position"/>
-                <state_interface name="velocity"/>
-                <state_interface name="effort"/>
-            </joint>
-            <joint name="joint_4">
-                <command_interface name="position"/>
-                <command_interface name="effort"/>
-                <state_interface name="position"/>
-                <state_interface name="velocity"/>
-                <state_interface name="effort"/>
-            </joint>
-            <joint name="joint_5">
-                <command_interface name="position"/>
-                <command_interface name="effort"/>
-                <state_interface name="position"/>
-                <state_interface name="velocity"/>
-                <state_interface name="effort"/>
-            </joint>
-            <joint name="joint_6">
-                <command_interface name="position"/>
-                <command_interface name="effort"/>
-                <state_interface name="position"/>
-                <state_interface name="velocity"/>
-                <state_interface name="effort"/>
-            </joint>
-        </ros2_control>
-    </xacro:if>
-    <xacro:unless value="$(arg sim_mode)">
-        <ros2_control name="REAL_SYSTEM" type="SYSTEM">
             <hardware>
                 <plugin>gazebo_ros2_control/GazeboSystem</plugin>
@@ -106,4 +53,101 @@
             </joint>
         </ros2_control>
+    </xacro:if>
+    <xacro:unless value="$(arg sim_mode)">
+        <ros2_control name="RealSystem" type="system">
+            <hardware>
+                <plugin>ethercat_driver/EthercatDriver</plugin>
+                <param name="master_id">0</param>
+                <param name="control_frequency">1000</param>
+            </hardware>
+            <joint name="joint_1">
+                <command_interface name="position"/>
+                <command_interface name="effort"/>
+                <!--            <command_interface name="velocity"/>-->
+                <!--            <command_interface name="effort"/>-->
+                <!--                <param name="min">-10</param>-->
+                <!--                <param name="max">10</param>-->
+                <state_interface name="position"/>
+                <state_interface name="velocity"/>
+                <state_interface name="effort"/>
+                <ec_module name="senso_joint_1">
+                    <plugin>ethercat_generic_plugins/EcSensoDrive</plugin>
+                    <param name="alias">0</param>
+                    <param name="position">0</param>
+                    <param name="mode_of_operation">8</param>
+                    <param name="slave_config">$(find sensorob)/config/joints_driver_config/senso_joint_1.yaml</param>
+                </ec_module>
+            </joint>
+            <joint name="joint_2">
+                <command_interface name="position"/>
+                <command_interface name="effort"/>
+                <state_interface name="position"/>
+                <state_interface name="velocity"/>
+                <state_interface name="effort"/>
+                <ec_module name="senso_joint_2">
+                    <plugin>ethercat_generic_plugins/EcSensoDrive</plugin>
+                    <param name="alias">0</param>
+                    <param name="position">0</param>
+                    <param name="mode_of_operation">8</param>
+                    <param name="slave_config">$(find sensorob)/config/joints_driver_config/senso_joint_2.yaml</param>
+                </ec_module>
+            </joint>
+            <joint name="joint_3">
+                <command_interface name="position"/>
+                <command_interface name="effort"/>
+                <state_interface name="position"/>
+                <state_interface name="velocity"/>
+                <state_interface name="effort"/>
+                <ec_module name="senso_joint_3">
+                    <plugin>ethercat_generic_plugins/EcSensoDrive</plugin>
+                    <param name="alias">0</param>
+                    <param name="position">0</param>
+                    <param name="mode_of_operation">8</param>
+                    <param name="slave_config">$(find sensorob)/config/joints_driver_config/senso_joint_3.yaml</param>
+                </ec_module>
+            </joint>
+            <joint name="joint_4">
+                <command_interface name="position"/>
+                <command_interface name="effort"/>
+                <state_interface name="position"/>
+                <state_interface name="velocity"/>
+                <state_interface name="effort"/>
+                <ec_module name="senso_joint_4">
+                    <plugin>ethercat_generic_plugins/EcSensoDrive</plugin>
+                    <param name="alias">0</param>
+                    <param name="position">0</param>
+                    <param name="mode_of_operation">8</param>
+                    <param name="slave_config">$(find sensorob)/config/joints_driver_config/senso_joint_4.yaml</param>
+                </ec_module>
+            </joint>
+            <joint name="joint_5">
+                <command_interface name="position"/>
+                <command_interface name="effort"/>
+                <state_interface name="position"/>
+                <state_interface name="velocity"/>
+                <state_interface name="effort"/>
+                <ec_module name="senso_joint_5">
+                    <plugin>ethercat_generic_plugins/EcSensoDrive</plugin>
+                    <param name="alias">0</param>
+                    <param name="position">0</param>
+                    <param name="mode_of_operation">8</param>
+                    <param name="slave_config">$(find sensorob)/config/joints_driver_config/senso_joint_5.yaml</param>
+                </ec_module>
+            </joint>
+            <joint name="joint_6">
+                <command_interface name="position"/>
+                <command_interface name="effort"/>
+                <state_interface name="position"/>
+                <state_interface name="velocity"/>
+                <state_interface name="effort"/>
+                <ec_module name="senso_joint_6">
+                    <plugin>ethercat_generic_plugins/EcSensoDrive</plugin>
+                    <param name="alias">0</param>
+                    <param name="position">0</param>
+                    <param name="mode_of_operation">8</param>
+                    <param name="slave_config">$(find sensorob)/config/joints_driver_config/senso_joint_6.yaml</param>
+                </ec_module>
+            </joint>
+        </ros2_control>
     </xacro:unless>
     <gazebo>

File: sensorob_description/urdf/sensorob.urdf (robot description, URDF)
Before this commit: robot sensorob, 8 links, 7 joints
Joints:
- joint joint_1: limit lower=-3.141592653589793 upper=3.141592653589793 effort=100 velocity=100 -> lower=-3.141592653589793 upper=3.141592653589793 effort=500 velocity=6
- joint joint_2: limit lower=-1.570796327 upper=1.570796327 effort=100 velocity=100 -> lower=-1.570796327 upper=1.570796327 effort=500 velocity=6
- joint joint_3: limit lower=-2.094395102 upper=2.094395102 effort=100 velocity=100 -> lower=-2.094395102 upper=2.094395102 effort=300 velocity=7
- joint joint_4: limit lower=-3.141592653589793 upper=3.141592653589793 effort=100 velocity=100 -> lower=-3.141592653589793 upper=3.141592653589793 effort=200 velocity=8
- joint joint_5: limit lower=-1.570796327 upper=1.570796327 effort=100 velocity=100 -> lower=-1.570796327 upper=1.570796327 effort=200 velocity=8
- joint joint_6: limit lower=-6.283185307 upper=6.283185307 effort=100 velocity=100 -> lower=-3.141592653589793 upper=3.141592653589793 effort=200 velocity=10

Commit message: fixes in robot_core + constraints in controllers

File: sensorob_description/urdf/robot_core.xacro (robot description, xacro)
@@ -155,5 +155,5 @@
     <child link="link_1"/>
     <axis xyz="0.0 -0.0 1.0"/>
-    <limit upper="3.141592653589793" lower="-3.141592653589793" effort="500" velocity="6"/> <!-- +-pi -->
+    <limit upper="3.1414" lower="-3.1414" effort="500" velocity="6"/> <!-- +-pi -->
   </joint>
   <joint name="joint_2" type="revolute">
@@ -176,5 +176,5 @@
     <child link="link_4"/>
     <axis xyz="0.0 0.0 1.0"/>
-    <limit upper="3.141592653589793" lower="-3.141592653589793" effort="200" velocity="8"/> <!-- +-pi -->
+    <limit upper="3.1414" lower="-3.1414" effort="200" velocity="8"/> <!-- +-pi -->
   </joint>
   <joint name="joint_5" type="revolute">
@@ -190,5 +190,5 @@
     <child link="link_6"/>
     <axis xyz="0.0 -0.0 -1.0"/>
-    <limit upper="3.141592653589793" lower="-3.141592653589793" effort="200" velocity="10"/> <!-- +-pi (cannot be higher because of an absolut encoder without flash disk)-->
+    <limit upper="3.1414" lower="-3.1414" effort="200" velocity="10"/> <!-- +-pi (cannot be higher because of an absolut encoder without flash disk)-->
   </joint>
 </robot>

File: sensorob_description/urdf/ros2_control.xacro (robot description, xacro)
@@ -98,6 +98,7 @@
                     <plugin>ethercat_generic_plugins/EcSensoDrive</plugin>
                     <param name="alias">0</param>
-                    <param name="position">0</param>
+                    <param name="position">5</param>
                     <param name="mode_of_operation">8</param>
+                    <param name="position_offset">-3.14159265359</param>
                     <param name="slave_config">$(find sensorob)/config/joints_driver_config/senso_joint_1.yaml</param>
                 </ec_module>
@@ -112,6 +113,7 @@
                     <plugin>ethercat_generic_plugins/EcSensoDrive</plugin>
                     <param name="alias">0</param>
-                    <param name="position">0</param>
+                    <param name="position">1</param>
                     <param name="mode_of_operation">8</param>
+                    <param name="position_offset">-3.14159265359</param>
                     <param name="slave_config">$(find sensorob)/config/joints_driver_config/senso_joint_2.yaml</param>
                 </ec_module>
@@ -126,6 +128,7 @@
                     <plugin>ethercat_generic_plugins/EcSensoDrive</plugin>
                     <param name="alias">0</param>
-                    <param name="position">0</param>
+                    <param name="position">2</param>
                     <param name="mode_of_operation">8</param>
+                    <param name="position_offset">-3.14159265359</param>
                     <param name="slave_config">$(find sensorob)/config/joints_driver_config/senso_joint_3.yaml</param>
                 </ec_module>
@@ -140,6 +143,7 @@
                     <plugin>ethercat_generic_plugins/EcSensoDrive</plugin>
                     <param name="alias">0</param>
-                    <param name="position">0</param>
+                    <param name="position">3</param>
                     <param name="mode_of_operation">8</param>
+                    <param name="position_offset">-3.14159265359</param>
                     <param name="slave_config">$(find sensorob)/config/joints_driver_config/senso_joint_4.yaml</param>
                 </ec_module>
@@ -154,6 +158,7 @@
                     <plugin>ethercat_generic_plugins/EcSensoDrive</plugin>
                     <param name="alias">0</param>
-                    <param name="position">0</param>
+                    <param name="position">4</param>
                     <param name="mode_of_operation">8</param>
+                    <param name="position_offset">-3.14159265359</param>
                     <param name="slave_config">$(find sensorob)/config/joints_driver_config/senso_joint_5.yaml</param>
                 </ec_module>
@@ -170,4 +175,5 @@
                     <param name="position">0</param>
                     <param name="mode_of_operation">8</param>
+                    <param name="position_offset">-3.14159265359</param>
                     <param name="slave_config">$(find sensorob)/config/joints_driver_config/senso_joint_6.yaml</param>
                 </ec_module>

Commit message: robot model updated

File: sensorob_description/urdf/robot_core.xacro (robot description, xacro)
@@ -146,5 +146,5 @@
   </link>
   <joint name="world_link_joint" type="fixed">
-    <origin xyz="0.05 0.05 0.2" rpy="0 0 0"/>
+    <origin xyz="-0.065 0.0 0.1328" rpy="0 0 0"/>
     <parent link="world"/>
     <child link="base_link"/>
@@ -189,5 +189,5 @@
     <parent link="link_5"/>
     <child link="link_6"/>
-    <axis xyz="0.0 -0.0 -1.0"/>
+    <axis xyz="0.0 -0.0 1.0"/>
     <limit upper="3.1414" lower="-3.1414" effort="200" velocity="10"/> <!-- +-pi (cannot be higher because of an absolut encoder without flash disk)-->
   </joint>

File: sensorob_description/urdf/sensorob.urdf (robot description, URDF)
Before this commit: robot sensorob, 8 links, 7 joints
Joints:
- joint joint_6: axis 0.0 -0.0 -1.0 -> 0.0 -0.0 11.0
- joint world_link_joint: origin xyz=0.05 0.05 0.2 rpy=0 0 0 -> xyz=-0.065 0.0 0.1328 rpy=0 0 0
