Commit message: robot model fixes

File: sensorob_description/urdf/robot_core.xacro (robot description, xacro)
@@ -150,4 +150,5 @@
     <child link="base_link"/>
   </joint>
+<!-- data from https://www.sensodrive.de/products/torque-technology-senso-joint.php#:~:text=requirements%20if%20necessary.-,Technical%20data,-Technical%20data%20SensoJoint -->
   <joint name="joint_1" type="revolute">
     <origin xyz="0.06828 0.001091 0.070444" rpy="0 0 0"/>
@@ -155,5 +156,6 @@
     <child link="link_1"/>
     <axis xyz="0.0 -0.0 1.0"/>
-    <limit upper="3.1414" lower="-3.1414" effort="500" velocity="6"/> <!-- +-pi -->
+    <limit upper="${pi}" lower="${-pi}" effort="52" velocity="1.6755"/> <!--drive 5012 52Nm, 16/min-1 -->
+    <dynamics damping="1.0" friction="0.5"/>  <!-- damping  [Nms/rad], friction [Nm]-->
   </joint>
   <joint name="joint_2" type="revolute">
@@ -162,5 +164,6 @@
     <child link="link_2"/>
     <axis xyz="-1.0 0.0 -0.0"/>
-    <limit upper="1.570796327" lower="-1.570796327" effort="500" velocity="6"/> <!-- +-pi/2 -->
+    <limit upper="${pi/2}" lower="${-pi/2}" effort="52" velocity="1.6755"/> <!--drive 5012 52Nm, 16/min-1 -->
+    <dynamics damping="1.0" friction="0.5"/>  <!-- damping  [Nms/rad], friction [Nm]-->
   </joint>
   <joint name="joint_3" type="revolute">
@@ -169,5 +172,6 @@
     <child link="link_3"/>
     <axis xyz="1.0 0.0 0.0"/>
-    <limit upper="2.094395102" lower="-2.094395102" effort="300" velocity="7"/> <!-- +-2pi/3-->
+    <limit upper="${2*pi/3}" lower="${-2*pi/3}" effort="24" velocity="1.9896"/> <!--drive 4010 24Nm, 19/min-1 -->
+    <dynamics damping="1.0" friction="0.5"/>  <!-- damping  [Nms/rad], friction [Nm]-->
   </joint>
   <joint name="joint_4" type="revolute">
@@ -176,5 +180,6 @@
     <child link="link_4"/>
     <axis xyz="0.0 0.0 1.0"/>
-    <limit upper="3.1414" lower="-3.1414" effort="200" velocity="8"/> <!-- +-pi -->
+    <limit upper="${pi}" lower="${-pi}" effort="7.8" velocity="2.5133"/> <!--drive 3008 7.8Nm, 24/min-1 -->
+    <dynamics damping="1.0" friction="0.5"/>  <!-- damping  [Nms/rad], friction [Nm]-->
   </joint>
   <joint name="joint_5" type="revolute">
@@ -183,5 +188,6 @@
     <child link="link_5"/>
     <axis xyz="-1.0 -0.0 0.0"/>
-    <limit upper="1.570796327" lower="-1.570796327" effort="200" velocity="8"/> <!-- +-pi/2 -->
+    <limit upper="${pi/2}" lower="${-pi/2}" effort="7.8" velocity="2.5133"/> <!--drive 3008 7.8Nm, 24/min-1 -->
+    <dynamics damping="1.0" friction="0.5"/>  <!-- damping  [Nms/rad], friction [Nm]-->
   </joint>
   <joint name="joint_6" type="revolute">
@@ -189,6 +195,7 @@
     <parent link="link_5"/>
     <child link="link_6"/>
-    <axis xyz="0.0 -0.0 -1.0"/>
-    <limit upper="3.1414" lower="-3.1414" effort="200" velocity="10"/> <!-- +-pi (cannot be higher because of an absolut encoder without flash disk)-->
+    <axis xyz="0.0 -0.0 1.0"/>
+    <limit upper="${pi}" lower="${-pi}" effort="7.8" velocity="2.5133"/> <!--drive 3008 7.8Nm, 24/min-1 -->
+    <dynamics damping="1.0" friction="0.5"/>  <!-- damping  [Nms/rad], friction [Nm]-->
   </joint>
 </robot>

Commit message: robot model edits

File: sensorob_description/urdf/robot_core.xacro (robot description, xacro)
@@ -150,4 +150,5 @@
     <child link="base_link"/>
   </joint>
+<!-- data from https://www.sensodrive.de/products/torque-technology-senso-joint.php#:~:text=requirements%20if%20necessary.-,Technical%20data,-Technical%20data%20SensoJoint -->
   <joint name="joint_1" type="revolute">
     <origin xyz="0.06828 0.001091 0.070444" rpy="0 0 0"/>
@@ -155,5 +156,6 @@
     <child link="link_1"/>
     <axis xyz="0.0 -0.0 1.0"/>
-    <limit upper="3.1414" lower="-3.1414" effort="500" velocity="6"/> <!-- +-pi -->
+    <limit upper="${pi}" lower="${-pi}" effort="52" velocity="1.6755"/> <!--drive 5012 52Nm, 16/min-1 -->
+    <dynamics damping="1.0" friction="0.5"/>  <!-- damping  [Nms/rad], friction [Nm]-->
   </joint>
   <joint name="joint_2" type="revolute">
@@ -162,5 +164,6 @@
     <child link="link_2"/>
     <axis xyz="-1.0 0.0 -0.0"/>
-    <limit upper="1.570796327" lower="-1.570796327" effort="500" velocity="6"/> <!-- +-pi/2 -->
+    <limit upper="${pi/2}" lower="${-pi/2}" effort="52" velocity="1.6755"/> <!--drive 5012 52Nm, 16/min-1 -->
+    <dynamics damping="1.0" friction="0.5"/>  <!-- damping  [Nms/rad], friction [Nm]-->
   </joint>
   <joint name="joint_3" type="revolute">
@@ -169,5 +172,6 @@
     <child link="link_3"/>
     <axis xyz="1.0 0.0 0.0"/>
-    <limit upper="2.094395102" lower="-2.094395102" effort="300" velocity="7"/> <!-- +-2pi/3-->
+    <limit upper="${2*pi/3}" lower="${-2*pi/3}" effort="24" velocity="1.9896"/> <!--drive 4010 24Nm, 19/min-1 -->
+    <dynamics damping="1.0" friction="0.5"/>  <!-- damping  [Nms/rad], friction [Nm]-->
   </joint>
   <joint name="joint_4" type="revolute">
@@ -176,5 +180,6 @@
     <child link="link_4"/>
     <axis xyz="0.0 0.0 1.0"/>
-    <limit upper="3.1414" lower="-3.1414" effort="200" velocity="8"/> <!-- +-pi -->
+    <limit upper="${pi}" lower="${-pi}" effort="7.8" velocity="2.5133"/> <!--drive 3008 7.8Nm, 24/min-1 -->
+    <dynamics damping="1.0" friction="0.5"/>  <!-- damping  [Nms/rad], friction [Nm]-->
   </joint>
   <joint name="joint_5" type="revolute">
@@ -183,5 +188,6 @@
     <child link="link_5"/>
     <axis xyz="-1.0 -0.0 0.0"/>
-    <limit upper="1.570796327" lower="-1.570796327" effort="200" velocity="8"/> <!-- +-pi/2 -->
+    <limit upper="${pi/2}" lower="${-pi/2}" effort="7.8" velocity="2.5133"/> <!--drive 3008 7.8Nm, 24/min-1 -->
+    <dynamics damping="1.0" friction="0.5"/>  <!-- damping  [Nms/rad], friction [Nm]-->
   </joint>
   <joint name="joint_6" type="revolute">
@@ -190,5 +196,6 @@
     <child link="link_6"/>
     <axis xyz="0.0 -0.0 1.0"/>
-    <limit upper="3.1414" lower="-3.1414" effort="200" velocity="10"/> <!-- +-pi (cannot be higher because of an absolut encoder without flash disk)-->
+    <limit upper="${pi}" lower="${-pi}" effort="7.8" velocity="2.5133"/> <!--drive 3008 7.8Nm, 24/min-1 -->
+    <dynamics damping="1.0" friction="0.5"/>  <!-- damping  [Nms/rad], friction [Nm]-->
   </joint>
 </robot>

File: sensorob_description/urdf/ros2_control.xacro (robot description, xacro)
@@ -98,5 +98,5 @@
                     <plugin>ethercat_generic_plugins/EcSensoDrive</plugin>
                     <param name="alias">0</param>
-                    <param name="position">5</param>
+                    <param name="position">2</param>
                     <param name="mode_of_operation">8</param>
                     <param name="position_offset">-3.14159265359</param>
@@ -113,5 +113,5 @@
                     <plugin>ethercat_generic_plugins/EcSensoDrive</plugin>
                     <param name="alias">0</param>
-                    <param name="position">1</param>
+                    <param name="position">3</param>
                     <param name="mode_of_operation">8</param>
                     <param name="position_offset">-3.14159265359</param>
@@ -128,5 +128,5 @@
                     <plugin>ethercat_generic_plugins/EcSensoDrive</plugin>
                     <param name="alias">0</param>
-                    <param name="position">2</param>
+                    <param name="position">4</param>
                     <param name="mode_of_operation">8</param>
                     <param name="position_offset">-3.14159265359</param>
@@ -143,5 +143,5 @@
                     <plugin>ethercat_generic_plugins/EcSensoDrive</plugin>
                     <param name="alias">0</param>
-                    <param name="position">3</param>
+                    <param name="position">0</param>
                     <param name="mode_of_operation">8</param>
                     <param name="position_offset">-3.14159265359</param>
@@ -158,5 +158,5 @@
                     <plugin>ethercat_generic_plugins/EcSensoDrive</plugin>
                     <param name="alias">0</param>
-                    <param name="position">4</param>
+                    <param name="position">5</param>
                     <param name="mode_of_operation">8</param>
                     <param name="position_offset">-3.14159265359</param>
@@ -173,5 +173,5 @@
                     <plugin>ethercat_generic_plugins/EcSensoDrive</plugin>
                     <param name="alias">0</param>
-                    <param name="position">0</param>
+                    <param name="position">1</param>
                     <param name="mode_of_operation">8</param>
                     <param name="position_offset">-3.14159265359</param>
@@ -185,4 +185,8 @@
             <parameters>$(find sensorob)/config/sensorob_controllers.yaml</parameters>
             <parameters>$(find sensorob)/config/gaz_ros2_ctl_use_sim.yaml</parameters>
+            <robot_param>robot_description</robot_param>
+            <robot_param_node>robot_state_publisher</robot_param_node>
+            <controller_manager_name>controller_manager</controller_manager_name>
+            <hold_joints>True</hold_joints>
         </plugin>
     </gazebo>

Commit message: links weight

File: sensorob_description/urdf/robot_core.xacro (robot description, xacro)
@@ -8,5 +8,5 @@
     <inertial>
       <origin xyz="0.0684293395086911 0.0009438578686822592 -0.026799613448182283" rpy="0 0 0"/>
-      <mass value="1.855542034998811"/>
+      <mass value="3.0"/>
       <inertia ixx="0.00951" iyy="0.008318" izz="0.007035" ixy="1e-05" iyz="-2.2e-05" ixz="2.3e-05"/>
     </inertial>
@@ -28,5 +28,5 @@
     <inertial>
       <origin xyz="-0.019055565879577983 0.00028607059109358383 0.0917034573021166" rpy="0 0 0"/>
-      <mass value="2.1673778446055563"/>
+      <mass value="3.0"/>
       <inertia ixx="0.006709" iyy="0.007067" izz="0.005681" ixy="-7e-05" iyz="-1.2e-05" ixz="0.000853"/>
     </inertial>
@@ -48,5 +48,5 @@
     <inertial>
       <origin xyz="-0.04019415358244136 -0.0010759815082800456 0.24369077827545405" rpy="0 0 0"/>
-      <mass value="3.7950516594171546"/>
+      <mass value="4.9"/>
       <inertia ixx="0.125698" iyy="0.115802" izz="0.018463" ixy="-8.3e-05" iyz="-6.5e-05" ixz="-0.001156"/>
     </inertial>
@@ -68,5 +68,5 @@
     <inertial>
       <origin xyz="0.03693926470328392 0.0001460307076859913 0.13201293251123314" rpy="0 0 0"/>
-      <mass value="1.1351525716942115"/>
+      <mass value="1.9"/>
       <inertia ixx="0.007232" iyy="0.006989" izz="0.001398" ixy="7e-06" iyz="6e-06" ixz="-7.5e-05"/>
     </inertial>
@@ -88,5 +88,5 @@
     <inertial>
       <origin xyz="0.037181058344095096 0.0001800805076532456 0.11081132606474708" rpy="0 0 0"/>
-      <mass value="1.2025016995467235"/>
+      <mass value="2.0"/>
       <inertia ixx="0.004084" iyy="0.004612" izz="0.002169" ixy="-1e-06" iyz="-1.3e-05" ixz="-0.000638"/>
     </inertial>
@@ -108,5 +108,5 @@
     <inertial>
       <origin xyz="-0.015451790870986186 -0.0004790673243593754 0.11721977365766034" rpy="0 0 0"/>
-      <mass value="1.10970553090912"/>
+      <mass value="1.85"/>
       <inertia ixx="0.006037" iyy="0.005961" izz="0.001491" ixy="9e-06" iyz="5e-06" ixz="-0.000401"/>
     </inertial>

Commit message: robot model
Updated submodule ethercat_driver_ros2

File: sensorob_description/urdf/robot_core.xacro (robot description, xacro)
@@ -156,5 +156,5 @@
     <child link="link_1"/>
     <axis xyz="0.0 -0.0 1.0"/>
-    <limit upper="${pi}" lower="${-pi}" effort="52" velocity="1.6755"/> <!--drive 5012 52Nm, 16/min-1 -->
+    <limit upper="${0.999493*pi}" lower="${-0.999493*pi}" effort="52" velocity="1.6755"/> <!--drive 5012 52Nm, 16/min-1 -->
     <dynamics damping="1.0" friction="0.5"/>  <!-- damping  [Nms/rad], friction [Nm]-->
   </joint>
@@ -180,5 +180,5 @@
     <child link="link_4"/>
     <axis xyz="0.0 0.0 1.0"/>
-    <limit upper="${pi}" lower="${-pi}" effort="7.8" velocity="2.5133"/> <!--drive 3008 7.8Nm, 24/min-1 -->
+    <limit upper="${0.999493*pi}" lower="${-0.999493*pi}" effort="7.8" velocity="2.5133"/> <!--drive 3008 7.8Nm, 24/min-1 -->
     <dynamics damping="1.0" friction="0.5"/>  <!-- damping  [Nms/rad], friction [Nm]-->
   </joint>
@@ -196,5 +196,5 @@
     <child link="link_6"/>
     <axis xyz="0.0 -0.0 1.0"/>
-    <limit upper="${pi}" lower="${-pi}" effort="7.8" velocity="2.5133"/> <!--drive 3008 7.8Nm, 24/min-1 -->
+    <limit upper="${0.999493*pi}" lower="${-0.999493*pi}" effort="7.8" velocity="2.5133"/> <!--drive 3008 7.8Nm, 24/min-1 -->
     <dynamics damping="1.0" friction="0.5"/>  <!-- damping  [Nms/rad], friction [Nm]-->
   </joint>

File: sensorob_description/urdf/ros2_control.xacro (robot description, xacro)
@@ -100,5 +100,5 @@
                     <param name="position">2</param>
                     <param name="mode_of_operation">8</param>
-                    <param name="position_offset">-3.14159265359</param>
+                    <param name="position_offset">-${pi}</param>
                     <param name="slave_config">$(find sensorob)/config/joints_driver_config/senso_joint_1.yaml</param>
                 </ec_module>
@@ -115,5 +115,5 @@
                     <param name="position">3</param>
                     <param name="mode_of_operation">8</param>
-                    <param name="position_offset">-3.14159265359</param>
+                    <param name="position_offset">-${pi}</param>
                     <param name="slave_config">$(find sensorob)/config/joints_driver_config/senso_joint_2.yaml</param>
                 </ec_module>
@@ -128,7 +128,7 @@
                     <plugin>ethercat_generic_plugins/EcSensoDrive</plugin>
                     <param name="alias">0</param>
-                    <param name="position">4</param>
+                    <param name="position">0</param>
                     <param name="mode_of_operation">8</param>
-                    <param name="position_offset">-3.14159265359</param>
+                    <param name="position_offset">-${pi}</param>
                     <param name="slave_config">$(find sensorob)/config/joints_driver_config/senso_joint_3.yaml</param>
                 </ec_module>
@@ -143,7 +143,7 @@
                     <plugin>ethercat_generic_plugins/EcSensoDrive</plugin>
                     <param name="alias">0</param>
-                    <param name="position">0</param>
+                    <param name="position">4</param>
                     <param name="mode_of_operation">8</param>
-                    <param name="position_offset">-3.14159265359</param>
+                    <param name="position_offset">-${pi}</param>
                     <param name="slave_config">$(find sensorob)/config/joints_driver_config/senso_joint_4.yaml</param>
                 </ec_module>
@@ -160,5 +160,5 @@
                     <param name="position">5</param>
                     <param name="mode_of_operation">8</param>
-                    <param name="position_offset">-3.14159265359</param>
+                    <param name="position_offset">-${pi}</param>
                     <param name="slave_config">$(find sensorob)/config/joints_driver_config/senso_joint_5.yaml</param>
                 </ec_module>
@@ -175,5 +175,5 @@
                     <param name="position">1</param>
                     <param name="mode_of_operation">8</param>
-                    <param name="position_offset">-3.14159265359</param>
+                    <param name="position_offset">-${pi}</param>
                     <param name="slave_config">$(find sensorob)/config/joints_driver_config/senso_joint_6.yaml</param>
                 </ec_module>
