Commit message: joint params to config file

File: sensorob_description/urdf/robot_core.xacro (robot description, xacro)
@@ -3,4 +3,5 @@
   <xacro:include filename="materials.xacro" />
   <xacro:include filename="sensorob.gazebo" />
+  <xacro:property name="jf" value="${xacro.load_yaml('$(find sensorob_description)/config/joint_parameters.yaml')}"/>
   <link name="world">
   </link>
@@ -150,5 +151,4 @@
     <child link="base_link"/>
   </joint>
-<!-- data from https://www.sensodrive.de/products/torque-technology-senso-joint.php#:~:text=requirements%20if%20necessary.-,Technical%20data,-Technical%20data%20SensoJoint -->
   <joint name="joint_1" type="revolute">
     <origin xyz="0.06828 0.001091 0.070444" rpy="0 0 0"/>
@@ -156,6 +156,6 @@
     <child link="link_1"/>
     <axis xyz="0.0 -0.0 1.0"/>
-    <limit upper="${0.999493*pi}" lower="${-0.999493*pi}" effort="52" velocity="1.6755"/> <!--drive 5012 52Nm, 16/min-1 -->
-    <dynamics damping="1.0" friction="0.5"/>  <!-- damping  [Nms/rad], friction [Nm]-->
+    <limit upper="${jf['joint_1']['upper']}" lower="${jf['joint_1']['lower']}" effort="${jf['joint_1']['effort']}" velocity="${jf['joint_1']['velocity']}"/>
+    <dynamics damping="${jf['joint_1']['dumping']}" friction="${jf['joint_1']['friction']}"/>
   </joint>
   <joint name="joint_2" type="revolute">
@@ -164,6 +164,6 @@
     <child link="link_2"/>
     <axis xyz="-1.0 0.0 -0.0"/>
-    <limit upper="${pi/2}" lower="${-pi/2}" effort="52" velocity="1.6755"/> <!--drive 5012 52Nm, 16/min-1 -->
-    <dynamics damping="1.0" friction="0.5"/>  <!-- damping  [Nms/rad], friction [Nm]-->
+    <limit upper="${jf['joint_2']['upper']}" lower="${jf['joint_2']['lower']}" effort="${jf['joint_2']['effort']}" velocity="${jf['joint_2']['velocity']}"/>
+    <dynamics damping="${jf['joint_2']['dumping']}" friction="${jf['joint_2']['friction']}"/>
   </joint>
   <joint name="joint_3" type="revolute">
@@ -172,6 +172,6 @@
     <child link="link_3"/>
     <axis xyz="1.0 0.0 0.0"/>
-    <limit upper="${2*pi/3}" lower="${-2*pi/3}" effort="24" velocity="1.9896"/> <!--drive 4010 24Nm, 19/min-1 -->
-    <dynamics damping="1.0" friction="0.5"/>  <!-- damping  [Nms/rad], friction [Nm]-->
+    <limit upper="${jf['joint_3']['upper']}" lower="${jf['joint_3']['lower']}" effort="${jf['joint_3']['effort']}" velocity="${jf['joint_3']['velocity']}"/>
+    <dynamics damping="${jf['joint_3']['dumping']}" friction="${jf['joint_3']['friction']}"/>
   </joint>
   <joint name="joint_4" type="revolute">
@@ -180,6 +180,6 @@
     <child link="link_4"/>
     <axis xyz="0.0 0.0 1.0"/>
-    <limit upper="${0.999493*pi}" lower="${-0.999493*pi}" effort="7.8" velocity="2.5133"/> <!--drive 3008 7.8Nm, 24/min-1 -->
-    <dynamics damping="1.0" friction="0.5"/>  <!-- damping  [Nms/rad], friction [Nm]-->
+    <limit upper="${jf['joint_4']['upper']}" lower="${jf['joint_4']['lower']}" effort="${jf['joint_4']['effort']}" velocity="${jf['joint_4']['velocity']}"/>
+    <dynamics damping="${jf['joint_4']['dumping']}" friction="${jf['joint_4']['friction']}"/>
   </joint>
   <joint name="joint_5" type="revolute">
@@ -188,6 +188,6 @@
     <child link="link_5"/>
     <axis xyz="-1.0 -0.0 0.0"/>
-    <limit upper="${pi/2}" lower="${-pi/2}" effort="7.8" velocity="2.5133"/> <!--drive 3008 7.8Nm, 24/min-1 -->
-    <dynamics damping="1.0" friction="0.5"/>  <!-- damping  [Nms/rad], friction [Nm]-->
+    <limit upper="${jf['joint_5']['upper']}" lower="${jf['joint_5']['lower']}" effort="${jf['joint_5']['effort']}" velocity="${jf['joint_5']['velocity']}"/>
+    <dynamics damping="${jf['joint_5']['dumping']}" friction="${jf['joint_5']['friction']}"/>
   </joint>
   <joint name="joint_6" type="revolute">
@@ -196,6 +196,6 @@
     <child link="link_6"/>
     <axis xyz="0.0 -0.0 1.0"/>
-    <limit upper="${0.999493*pi}" lower="${-0.999493*pi}" effort="7.8" velocity="2.5133"/> <!--drive 3008 7.8Nm, 24/min-1 -->
-    <dynamics damping="1.0" friction="0.5"/>  <!-- damping  [Nms/rad], friction [Nm]-->
+    <limit upper="${jf['joint_6']['upper']}" lower="${jf['joint_6']['lower']}" effort="${jf['joint_6']['effort']}" velocity="${jf['joint_6']['velocity']}"/>
+    <dynamics damping="${jf['joint_6']['dumping']}" friction="${jf['joint_6']['friction']}"/>
   </joint>
 </robot>

File: sensorob_description/urdf/ros2_control.xacro (robot description, xacro)
@@ -1,4 +1,5 @@
 <?xml version="1.0" ?>
 <robot xmlns:xacro="http://www.ros.org/wiki/xacro" >
+<xacro:property name="jf" value="${xacro.load_yaml('$(find sensorob_description)/config/joint_parameters.yaml')}"/>
     <xacro:if value="$(arg sim_mode)">
         <ros2_control name="GazeboSystem" type="system">
@@ -14,8 +15,8 @@
                 <!--                <param name="max">10</param>-->
                 <state_interface name="position">
-                    <param name="initial_value">0.0</param>
+                    <param name="initial_value">${jf['joint_1']['init_pos']}</param>
                 </state_interface>
                 <state_interface name="velocity">
-                    <param name="initial_value">0.0</param>
+                    <param name="initial_value">${jf['joint_1']['init_vel']}</param>
                 </state_interface>
                 <state_interface name="effort"/>
@@ -25,8 +26,8 @@
                 <command_interface name="effort"/>
                 <state_interface name="position">
-                    <param name="initial_value">0.0</param>
+                    <param name="initial_value">${jf['joint_2']['init_pos']}</param>
                 </state_interface>
                 <state_interface name="velocity">
-                    <param name="initial_value">0.0</param>
+                    <param name="initial_value">${jf['joint_2']['init_vel']}</param>
                 </state_interface>
                 <state_interface name="effort"/>
@@ -36,8 +37,8 @@
                 <command_interface name="effort"/>
                 <state_interface name="position">
-                    <param name="initial_value">0.0</param>
+                    <param name="initial_value">${jf['joint_3']['init_pos']}</param>
                 </state_interface>
                 <state_interface name="velocity">
-                    <param name="initial_value">0.0</param>
+                    <param name="initial_value">${jf['joint_3']['init_vel']}</param>
                 </state_interface>
                 <state_interface name="effort"/>
@@ -47,8 +48,8 @@
                 <command_interface name="effort"/>
                 <state_interface name="position">
-                    <param name="initial_value">0.0</param>
+                    <param name="initial_value">${jf['joint_4']['init_pos']}</param>
                 </state_interface>
                 <state_interface name="velocity">
-                    <param name="initial_value">0.0</param>
+                    <param name="initial_value">${jf['joint_4']['init_vel']}</param>
                 </state_interface>
                 <state_interface name="effort"/>
@@ -58,8 +59,8 @@
                 <command_interface name="effort"/>
                 <state_interface name="position">
-                    <param name="initial_value">0.0</param>
+                    <param name="initial_value">${jf['joint_5']['init_pos']}</param>
                 </state_interface>
                 <state_interface name="velocity">
-                    <param name="initial_value">0.0</param>
+                    <param name="initial_value">${jf['joint_5']['init_vel']}</param>
                 </state_interface>
                 <state_interface name="effort"/>
@@ -69,8 +70,8 @@
                 <command_interface name="effort"/>
                 <state_interface name="position">
-                    <param name="initial_value">0.0</param>
+                    <param name="initial_value">${jf['joint_6']['init_pos']}</param>
                 </state_interface>
                 <state_interface name="velocity">
-                    <param name="initial_value">0.0</param>
+                    <param name="initial_value">${jf['joint_6']['init_vel']}</param>
                 </state_interface>
                 <state_interface name="effort"/>

Commit message: joint update

File: sensorob_description/urdf/robot_core.xacro (robot description, xacro)
@@ -155,5 +155,5 @@
     <parent link="base_link"/>
     <child link="link_1"/>
-    <axis xyz="0.0 -0.0 1.0"/>
+    <axis xyz="0.0 -0.0 -1.0"/>
     <limit upper="${jf['joint_1']['upper']}" lower="${jf['joint_1']['lower']}" effort="${jf['joint_1']['effort']}" velocity="${jf['joint_1']['velocity']}"/>
     <dynamics damping="${jf['joint_1']['dumping']}" friction="${jf['joint_1']['friction']}"/>
@@ -163,5 +163,5 @@
     <parent link="link_1"/>
     <child link="link_2"/>
-    <axis xyz="-1.0 0.0 -0.0"/>
+    <axis xyz="1.0 0.0 -0.0"/>
     <limit upper="${jf['joint_2']['upper']}" lower="${jf['joint_2']['lower']}" effort="${jf['joint_2']['effort']}" velocity="${jf['joint_2']['velocity']}"/>
     <dynamics damping="${jf['joint_2']['dumping']}" friction="${jf['joint_2']['friction']}"/>
@@ -171,5 +171,5 @@
     <parent link="link_2"/>
     <child link="link_3"/>
-    <axis xyz="1.0 0.0 0.0"/>
+    <axis xyz="-1.0 0.0 0.0"/>
     <limit upper="${jf['joint_3']['upper']}" lower="${jf['joint_3']['lower']}" effort="${jf['joint_3']['effort']}" velocity="${jf['joint_3']['velocity']}"/>
     <dynamics damping="${jf['joint_3']['dumping']}" friction="${jf['joint_3']['friction']}"/>
@@ -179,5 +179,5 @@
     <parent link="link_3"/>
     <child link="link_4"/>
-    <axis xyz="0.0 0.0 1.0"/>
+    <axis xyz="0.0 0.0 -1.0"/>
     <limit upper="${jf['joint_4']['upper']}" lower="${jf['joint_4']['lower']}" effort="${jf['joint_4']['effort']}" velocity="${jf['joint_4']['velocity']}"/>
     <dynamics damping="${jf['joint_4']['dumping']}" friction="${jf['joint_4']['friction']}"/>
@@ -187,5 +187,5 @@
     <parent link="link_4"/>
     <child link="link_5"/>
-    <axis xyz="-1.0 -0.0 0.0"/>
+    <axis xyz="1.0 -0.0 0.0"/>
     <limit upper="${jf['joint_5']['upper']}" lower="${jf['joint_5']['lower']}" effort="${jf['joint_5']['effort']}" velocity="${jf['joint_5']['velocity']}"/>
     <dynamics damping="${jf['joint_5']['dumping']}" friction="${jf['joint_5']['friction']}"/>
@@ -195,5 +195,5 @@
     <parent link="link_5"/>
     <child link="link_6"/>
-    <axis xyz="0.0 -0.0 1.0"/>
+    <axis xyz="0.0 -0.0 -1.0"/>
     <limit upper="${jf['joint_6']['upper']}" lower="${jf['joint_6']['lower']}" effort="${jf['joint_6']['effort']}" velocity="${jf['joint_6']['velocity']}"/>
     <dynamics damping="${jf['joint_6']['dumping']}" friction="${jf['joint_6']['friction']}"/>

File: sensorob_description/urdf/ros2_control.xacro (robot description, xacro)
@@ -99,5 +99,5 @@
                     <plugin>ethercat_generic_plugins/EcSensoDrive</plugin>
                     <param name="alias">0</param>
-                    <param name="position">2</param>
+                    <param name="position">0</param>
                     <param name="mode_of_operation">8</param>
                     <param name="position_offset">-${pi}</param>
@@ -114,5 +114,5 @@
                     <plugin>ethercat_generic_plugins/EcSensoDrive</plugin>
                     <param name="alias">0</param>
-                    <param name="position">3</param>
+                    <param name="position">1</param>
                     <param name="mode_of_operation">8</param>
                     <param name="position_offset">-${pi}</param>
@@ -129,5 +129,5 @@
                     <plugin>ethercat_generic_plugins/EcSensoDrive</plugin>
                     <param name="alias">0</param>
-                    <param name="position">0</param>
+                    <param name="position">2</param>
                     <param name="mode_of_operation">8</param>
                     <param name="position_offset">-${pi}</param>
@@ -144,5 +144,5 @@
                     <plugin>ethercat_generic_plugins/EcSensoDrive</plugin>
                     <param name="alias">0</param>
-                    <param name="position">4</param>
+                    <param name="position">3</param>
                     <param name="mode_of_operation">8</param>
                     <param name="position_offset">-${pi}</param>
@@ -159,5 +159,5 @@
                     <plugin>ethercat_generic_plugins/EcSensoDrive</plugin>
                     <param name="alias">0</param>
-                    <param name="position">5</param>
+                    <param name="position">4</param>
                     <param name="mode_of_operation">8</param>
                     <param name="position_offset">-${pi}</param>
@@ -174,5 +174,5 @@
                     <plugin>ethercat_generic_plugins/EcSensoDrive</plugin>
                     <param name="alias">0</param>
-                    <param name="position">1</param>
+                    <param name="position">5</param>
                     <param name="mode_of_operation">8</param>
                     <param name="position_offset">-${pi}</param>
