Commit message: sim_mode propagated

File: sensorob_description/urdf/ros2_control.xacro (robot description, xacro)
@@ -1,58 +1,114 @@
 <?xml version="1.0" ?>
 <robot xmlns:xacro="http://www.ros.org/wiki/xacro" >
-    <ros2_control name="GazeboSystem" type="system">
-        <hardware>
-            <plugin>gazebo_ros2_control/GazeboSystem</plugin>
-        </hardware>
-        <joint name="joint_1">
-            <command_interface name="position"/>
-            <command_interface name="effort"/>
-<!--            <command_interface name="velocity"/>-->
-<!--            <command_interface name="effort"/>-->
-<!--                <param name="min">-10</param>-->
-<!--                <param name="max">10</param>-->
-            <state_interface name="position"/>
-            <state_interface name="velocity"/>
-            <state_interface name="effort"/>
-        </joint>
-        <joint name="joint_2">
-            <command_interface name="position"/>
-            <command_interface name="effort"/>
-            <state_interface name="position"/>
-            <state_interface name="velocity"/>
-            <state_interface name="effort"/>
-        </joint>
-        <joint name="joint_3">
-            <command_interface name="position"/>
-            <command_interface name="effort"/>
-            <state_interface name="position"/>
-            <state_interface name="velocity"/>
-            <state_interface name="effort"/>
-        </joint>
-        <joint name="joint_4">
-            <command_interface name="position"/>
-            <command_interface name="effort"/>
-            <state_interface name="position"/>
-            <state_interface name="velocity"/>
-            <state_interface name="effort"/>
-        </joint>
-        <joint name="joint_5">
-            <command_interface name="position"/>
-            <command_interface name="effort"/>
-            <state_interface name="position"/>
-            <state_interface name="velocity"/>
-            <state_interface name="effort"/>
-        </joint>
-        <joint name="joint_6">
-            <command_interface name="position"/>
-            <command_interface name="effort"/>
-            <state_interface name="position"/>
-            <state_interface name="velocity"/>
-            <state_interface name="effort"/>
-        </joint>
-    </ros2_control>
+    <xacro:if value="$(arg sim_mode)">
+        <ros2_control name="GazeboSystem" type="system">
+            <hardware>
+                <plugin>gazebo_ros2_control/GazeboSystem</plugin>
+            </hardware>
+            <joint name="joint_1">
+                <command_interface name="position"/>
+                <command_interface name="effort"/>
+    <!--            <command_interface name="velocity"/>-->
+    <!--            <command_interface name="effort"/>-->
+    <!--                <param name="min">-10</param>-->
+    <!--                <param name="max">10</param>-->
+                <state_interface name="position"/>
+                <state_interface name="velocity"/>
+                <state_interface name="effort"/>
+            </joint>
+            <joint name="joint_2">
+                <command_interface name="position"/>
+                <command_interface name="effort"/>
+                <state_interface name="position"/>
+                <state_interface name="velocity"/>
+                <state_interface name="effort"/>
+            </joint>
+            <joint name="joint_3">
+                <command_interface name="position"/>
+                <command_interface name="effort"/>
+                <state_interface name="position"/>
+                <state_interface name="velocity"/>
+                <state_interface name="effort"/>
+            </joint>
+            <joint name="joint_4">
+                <command_interface name="position"/>
+                <command_interface name="effort"/>
+                <state_interface name="position"/>
+                <state_interface name="velocity"/>
+                <state_interface name="effort"/>
+            </joint>
+            <joint name="joint_5">
+                <command_interface name="position"/>
+                <command_interface name="effort"/>
+                <state_interface name="position"/>
+                <state_interface name="velocity"/>
+                <state_interface name="effort"/>
+            </joint>
+            <joint name="joint_6">
+                <command_interface name="position"/>
+                <command_interface name="effort"/>
+                <state_interface name="position"/>
+                <state_interface name="velocity"/>
+                <state_interface name="effort"/>
+            </joint>
+        </ros2_control>
+    </xacro:if>
+    <xacro:unless value="$(arg sim_mode)">
+        <ros2_control name="REAL_SYSTEM" type="SYSTEM">
+            <hardware>
+                <plugin>gazebo_ros2_control/GazeboSystem</plugin>
+            </hardware>
+            <joint name="joint_1">
+                <command_interface name="position"/>
+                <command_interface name="effort"/>
+                <!--            <command_interface name="velocity"/>-->
+                <!--            <command_interface name="effort"/>-->
+                <!--                <param name="min">-10</param>-->
+                <!--                <param name="max">10</param>-->
+                <state_interface name="position"/>
+                <state_interface name="velocity"/>
+                <state_interface name="effort"/>
+            </joint>
+            <joint name="joint_2">
+                <command_interface name="position"/>
+                <command_interface name="effort"/>
+                <state_interface name="position"/>
+                <state_interface name="velocity"/>
+                <state_interface name="effort"/>
+            </joint>
+            <joint name="joint_3">
+                <command_interface name="position"/>
+                <command_interface name="effort"/>
+                <state_interface name="position"/>
+                <state_interface name="velocity"/>
+                <state_interface name="effort"/>
+            </joint>
+            <joint name="joint_4">
+                <command_interface name="position"/>
+                <command_interface name="effort"/>
+                <state_interface name="position"/>
+                <state_interface name="velocity"/>
+                <state_interface name="effort"/>
+            </joint>
+            <joint name="joint_5">
+                <command_interface name="position"/>
+                <command_interface name="effort"/>
+                <state_interface name="position"/>
+                <state_interface name="velocity"/>
+                <state_interface name="effort"/>
+            </joint>
+            <joint name="joint_6">
+                <command_interface name="position"/>
+                <command_interface name="effort"/>
+                <state_interface name="position"/>
+                <state_interface name="velocity"/>
+                <state_interface name="effort"/>
+            </joint>
+        </ros2_control>
+    </xacro:unless>
     <gazebo>
         <plugin name="gazebo_ros2_control" filename="libgazebo_ros2_control.so">
             <parameters>$(find sensorob)/config/sensorob_controllers.yaml</parameters>
+            <parameters>$(find sensorob)/config/gaz_ros2_ctl_use_sim.yaml</parameters>
         </plugin>
     </gazebo>

Commit message: controller edits + added advanced config for joint6

File: sensorob_description/urdf/ros2_control.xacro (robot description, xacro)
@@ -88,4 +88,5 @@
             <joint name="joint_1">
                 <command_interface name="position"/>
+                <command_interface name="velocity"/>
                 <command_interface name="effort"/>
                 <!--            <command_interface name="velocity"/>-->
@@ -99,83 +100,88 @@
                     <plugin>ethercat_generic_plugins/EcSensoDrive</plugin>
                     <param name="alias">0</param>
+                    <param name="position">5</param>
+                    <param name="mode_of_operation">8</param>
+                    <param name="position_offset">-${pi}</param>
+                    <param name="slave_config">$(find sensorob)/config/joints_driver_config/senso_joint_1.yaml</param>
+                </ec_module>
+            </joint>
+            <joint name="joint_2">
+                <command_interface name="position"/>
+                <command_interface name="velocity"/>
+                <command_interface name="effort"/>
+                <state_interface name="position"/>
+                <state_interface name="velocity"/>
+                <state_interface name="effort"/>
+                <ec_module name="senso_joint_2">
+                    <plugin>ethercat_generic_plugins/EcSensoDrive</plugin>
+                    <param name="alias">0</param>
+                    <param name="position">1</param>
+                    <param name="mode_of_operation">8</param>
+                    <param name="position_offset">-${pi}</param>
+                    <param name="slave_config">$(find sensorob)/config/joints_driver_config/senso_joint_2.yaml</param>
+                </ec_module>
+            </joint>
+            <joint name="joint_3">
+                <command_interface name="position"/>
+                <command_interface name="velocity"/>
+                <command_interface name="effort"/>
+                <state_interface name="position"/>
+                <state_interface name="velocity"/>
+                <state_interface name="effort"/>
+                <ec_module name="senso_joint_3">
+                    <plugin>ethercat_generic_plugins/EcSensoDrive</plugin>
+                    <param name="alias">0</param>
+                    <param name="position">2</param>
+                    <param name="mode_of_operation">8</param>
+                    <param name="position_offset">-${pi}</param>
+                    <param name="slave_config">$(find sensorob)/config/joints_driver_config/senso_joint_3.yaml</param>
+                </ec_module>
+            </joint>
+            <joint name="joint_4">
+                <command_interface name="position"/>
+                <command_interface name="velocity"/>
+                <command_interface name="effort"/>
+                <state_interface name="position"/>
+                <state_interface name="velocity"/>
+                <state_interface name="effort"/>
+                <ec_module name="senso_joint_4">
+                    <plugin>ethercat_generic_plugins/EcSensoDrive</plugin>
+                    <param name="alias">0</param>
+                    <param name="position">3</param>
+                    <param name="mode_of_operation">8</param>
+                    <param name="position_offset">-${pi}</param>
+                    <param name="slave_config">$(find sensorob)/config/joints_driver_config/senso_joint_4.yaml</param>
+                </ec_module>
+            </joint>
+            <joint name="joint_5">
+                <command_interface name="position"/>
+                <command_interface name="velocity"/>
+                <command_interface name="effort"/>
+                <state_interface name="position"/>
+                <state_interface name="velocity"/>
+                <state_interface name="effort"/>
+                <ec_module name="senso_joint_5">
+                    <plugin>ethercat_generic_plugins/EcSensoDrive</plugin>
+                    <param name="alias">0</param>
+                    <param name="position">4</param>
+                    <param name="mode_of_operation">8</param>
+                    <param name="position_offset">-${pi}</param>
+                    <param name="slave_config">$(find sensorob)/config/joints_driver_config/senso_joint_5.yaml</param>
+                </ec_module>
+            </joint>
+            <joint name="joint_6">
+                <command_interface name="position"/>
+                <command_interface name="velocity"/>
+                <command_interface name="effort"/>
+                <state_interface name="position"/>
+                <state_interface name="velocity"/>
+                <state_interface name="effort"/>
+                <ec_module name="senso_joint_6">
+                    <plugin>ethercat_generic_plugins/EcSensoDrive</plugin>
+                    <param name="alias">0</param>
                     <param name="position">0</param>
-                    <param name="mode_of_operation">8</param>
-                    <param name="position_offset">-${pi}</param>
-                    <param name="slave_config">$(find sensorob)/config/joints_driver_config/senso_joint_1.yaml</param>
-                </ec_module>
-            </joint>
-            <joint name="joint_2">
-                <command_interface name="position"/>
-                <command_interface name="effort"/>
-                <state_interface name="position"/>
-                <state_interface name="velocity"/>
-                <state_interface name="effort"/>
-                <ec_module name="senso_joint_2">
-                    <plugin>ethercat_generic_plugins/EcSensoDrive</plugin>
-                    <param name="alias">0</param>
-                    <param name="position">1</param>
-                    <param name="mode_of_operation">8</param>
-                    <param name="position_offset">-${pi}</param>
-                    <param name="slave_config">$(find sensorob)/config/joints_driver_config/senso_joint_2.yaml</param>
-                </ec_module>
-            </joint>
-            <joint name="joint_3">
-                <command_interface name="position"/>
-                <command_interface name="effort"/>
-                <state_interface name="position"/>
-                <state_interface name="velocity"/>
-                <state_interface name="effort"/>
-                <ec_module name="senso_joint_3">
-                    <plugin>ethercat_generic_plugins/EcSensoDrive</plugin>
-                    <param name="alias">0</param>
-                    <param name="position">2</param>
-                    <param name="mode_of_operation">8</param>
-                    <param name="position_offset">-${pi}</param>
-                    <param name="slave_config">$(find sensorob)/config/joints_driver_config/senso_joint_3.yaml</param>
-                </ec_module>
-            </joint>
-            <joint name="joint_4">
-                <command_interface name="position"/>
-                <command_interface name="effort"/>
-                <state_interface name="position"/>
-                <state_interface name="velocity"/>
-                <state_interface name="effort"/>
-                <ec_module name="senso_joint_4">
-                    <plugin>ethercat_generic_plugins/EcSensoDrive</plugin>
-                    <param name="alias">0</param>
-                    <param name="position">3</param>
-                    <param name="mode_of_operation">8</param>
-                    <param name="position_offset">-${pi}</param>
-                    <param name="slave_config">$(find sensorob)/config/joints_driver_config/senso_joint_4.yaml</param>
-                </ec_module>
-            </joint>
-            <joint name="joint_5">
-                <command_interface name="position"/>
-                <command_interface name="effort"/>
-                <state_interface name="position"/>
-                <state_interface name="velocity"/>
-                <state_interface name="effort"/>
-                <ec_module name="senso_joint_5">
-                    <plugin>ethercat_generic_plugins/EcSensoDrive</plugin>
-                    <param name="alias">0</param>
-                    <param name="position">4</param>
-                    <param name="mode_of_operation">8</param>
-                    <param name="position_offset">-${pi}</param>
-                    <param name="slave_config">$(find sensorob)/config/joints_driver_config/senso_joint_5.yaml</param>
-                </ec_module>
-            </joint>
-            <joint name="joint_6">
-                <command_interface name="position"/>
-                <command_interface name="effort"/>
-                <state_interface name="position"/>
-                <state_interface name="velocity"/>
-                <state_interface name="effort"/>
-                <ec_module name="senso_joint_6">
-                    <plugin>ethercat_generic_plugins/EcSensoDrive</plugin>
-                    <param name="alias">0</param>
-                    <param name="position">5</param>
-                    <param name="mode_of_operation">8</param>
-                    <param name="position_offset">-${pi}</param>
-                    <param name="slave_config">$(find sensorob)/config/joints_driver_config/senso_joint_6.yaml</param>
+                    <param name="mode_of_operation">-108</param>
+                    <param name="position_offset">-${pi}</param>
+                    <param name="slave_config">$(find sensorob)/config/joints_driver_config/senso_joint_6_advanced.yaml</param>
                 </ec_module>
             </joint>

Commit message: tmp

File: sensorob_description/urdf/ros2_control.xacro (robot description, xacro)
@@ -98,5 +98,4 @@
                     <param name="position">0</param>
                     <param name="mode_of_operation">-108</param>
-                    <!-- <param name="position_offset">-${0}</param> -->
                     <param name="slave_config">$(find sensorob)/config/joints_driver_config/senso_joint_1_advanced.yaml</param>
                 </ec_module>
@@ -114,5 +113,4 @@
                     <param name="position">1</param>
                     <param name="mode_of_operation">-108</param>
-                    <!-- <param name="position_offset">-${0}</param> -->
                     <param name="slave_config">$(find sensorob)/config/joints_driver_config/senso_joint_2_advanced.yaml</param>
                 </ec_module>
@@ -130,5 +128,4 @@
                     <param name="position">2</param>
                     <param name="mode_of_operation">-108</param>
-                    <!-- <param name="position_offset">-${0}</param> -->
                     <param name="slave_config">$(find sensorob)/config/joints_driver_config/senso_joint_3_advanced.yaml</param>
                 </ec_module>
@@ -146,5 +143,4 @@
                     <param name="position">3</param>
                     <param name="mode_of_operation">-108</param>
-                    <!-- <param name="position_offset">-${0}</param> -->
                     <param name="slave_config">$(find sensorob)/config/joints_driver_config/senso_joint_4_advanced.yaml</param>
                 </ec_module>
@@ -162,5 +158,4 @@
                     <param name="position">4</param>
                     <param name="mode_of_operation">-108</param>
-                    <!-- <param name="position_offset">-${0}</param> -->
                     <param name="slave_config">$(find sensorob)/config/joints_driver_config/senso_joint_5_advanced.yaml</param>
                 </ec_module>
@@ -178,5 +173,4 @@
                     <param name="position">5</param>
                     <param name="mode_of_operation">-108</param>
-                    <!-- <param name="position_offset">-${0}</param> -->
                     <param name="slave_config">$(find sensorob)/config/joints_driver_config/senso_joint_6_advanced.yaml</param>
                 </ec_module>

File: sensorob_description/urdf/sensorob.urdf (robot description, URDF)
Before this commit: robot sensorob, 8 links, 7 joints
Joints:
- joint joint_1: axis 0.0 -0.0 1.0 -> 0.0 -0.0 -1.0
- joint joint_2: axis -1.0 0.0 -0.0 -> 1.0 0.0 -0.0
- joint joint_3: axis 1.0 0.0 0.0 -> -1.0 0.0 0.0
- joint joint_4: axis 0.0 0.0 1.0 -> 0.0 0.0 -1.0
- joint joint_5: axis -1.0 -0.0 0.0 -> 1.0 -0.0 0.0
- joint joint_6: axis 0.0 -0.0 11.0 -> 0.0 -0.0 -1.0; limit lower=-3.141592653589793 upper=3.141592653589793 effort=200 velocity=10 -> lower=-3.121592653589793 upper=3.121592653589793 effort=200 velocity=10
- joint world_link_joint: origin xyz=-0.065 0.0 0.1328 rpy=0 0 0 -> xyz=0.06828 0.001091 0.070444 rpy=0 0 0
