Commit message: ik edits

File: sensorob_description/urdf/sensorob.urdf (robot description, URDF)
Before this commit: robot sensorob, 8 links, 7 joints
Joints:
- joint joint_1: limit lower=-3.141592653589793 upper=3.141592653589793 effort=500 velocity=6 -> lower=-1.05 upper=1.05 effort=500 velocity=0.65
- joint joint_2: limit lower=-1.570796327 upper=1.570796327 effort=500 velocity=6 -> lower=-1.22 upper=1.22 effort=500 velocity=0.65
- joint joint_3: limit lower=-2.094395102 upper=2.094395102 effort=300 velocity=7 -> lower=-1.3 upper=1.3 effort=300 velocity=0.8
- joint joint_4: limit lower=-3.141592653589793 upper=3.141592653589793 effort=200 velocity=8 -> lower=-1.57 upper=1.57 effort=200 velocity=1
- joint joint_5: limit lower=-1.570796327 upper=1.570796327 effort=200 velocity=8 -> lower=-1.570796327 upper=1.570796327 effort=200 velocity=1
- joint joint_6: limit lower=-3.121592653589793 upper=3.121592653589793 effort=200 velocity=10 -> lower=-3.121592653589793 upper=3.121592653589793 effort=200 velocity=1
