Commit message: fake controllers

File: sensorob_moveit_config/config/sensorob.ros2_control.xacro (robot description, xacro)
@@ -1,6 +1,5 @@
 <?xml version="1.0"?>
 <robot xmlns:xacro="http://www.ros.org/wiki/xacro">
-    <xacro:macro name="sensorob_ros2_control" params="name initial_positions_file">
-        <xacro:property name="initial_positions" value="${load_yaml(initial_positions_file)['initial_positions']}"/>
+    <xacro:macro name="sensorob_ros2_control" params="name">
         <ros2_control name="${name}" type="system">
             <hardware>
@@ -11,5 +10,5 @@
                 <command_interface name="position"/>
                 <state_interface name="position">
-                  <param name="initial_value">${initial_positions['joint_1']}</param>
+                  <param name="initial_value">0.0</param>
                 </state_interface>
                 <state_interface name="velocity"/>
@@ -18,5 +17,5 @@
                 <command_interface name="position"/>
                 <state_interface name="position">
-                  <param name="initial_value">${initial_positions['joint_2']}</param>
+                  <param name="initial_value">0.0</param>
                 </state_interface>
                 <state_interface name="velocity"/>
@@ -25,5 +24,5 @@
                 <command_interface name="position"/>
                 <state_interface name="position">
-                  <param name="initial_value">${initial_positions['joint_3']}</param>
+                  <param name="initial_value">0.0</param>
                 </state_interface>
                 <state_interface name="velocity"/>
@@ -32,5 +31,5 @@
                 <command_interface name="position"/>
                 <state_interface name="position">
-                  <param name="initial_value">${initial_positions['joint_4']}</param>
+                  <param name="initial_value">0.0</param>
                 </state_interface>
                 <state_interface name="velocity"/>
@@ -39,5 +38,5 @@
                 <command_interface name="position"/>
                 <state_interface name="position">
-                  <param name="initial_value">${initial_positions['joint_5']}</param>
+                  <param name="initial_value">0.0</param>
                 </state_interface>
                 <state_interface name="velocity"/>
@@ -46,5 +45,5 @@
                 <command_interface name="position"/>
                 <state_interface name="position">
-                  <param name="initial_value">${initial_positions['joint_6']}</param>
+                  <param name="initial_value">0.0</param>
                 </state_interface>
                 <state_interface name="velocity"/>

File: sensorob_moveit_config/config/sensorob.urdf.xacro (robot description, xacro)
@@ -2,4 +2,5 @@
 <robot name="sensorob" xmlns:xacro="http://www.ros.org/wiki/xacro">
   <xacro:include filename="$(find sensorob_description)/urdf/robot_core.xacro" />
-  <xacro:include filename="$(find sensorob_description)/urdf/ros2_control.xacro" />
+   <xacro:include filename="sensorob.ros2_control.xacro" />
+   <xacro:sensorob_ros2_control name="FakeSystem"/>
 </robot>
